File: Eagle Projekt/Hardware-Neuron v2/Hardware-Neuron.brd (EAGLE design)
At the start: 160 x 100 mm, 54 parts, among them IC1 74LVC1G125DBV, IC2 74LVC1G125DBV, IC5 74AHC1G14DCK, Q10 FDN360P, Q11 FDN360P, Q17 BSS123, Q18 BSS123, Q19 FDN360P, Q20 FDN360P, Q21 FDN360P, Q22 FDN360P, Q23 FDN360P, Q24 FDN360P, Q25 FDN360P, Q26 FDN360P, Q5 FDN360P, Q6 BSS123, Q62 FDN360P, Q63 FDN360P, Q64 FDN360P, Q65 BSS123, Q66 BSS123, Q7 FDN360P, Q8 FDN360P, Q9 FDN360P

Commit message: updated v2
Parts:
- removed Q17, Q18: BSS123, transistor-small-signal:SOT23
- removed Q19, Q20, Q21, Q22: FDN360P, transistor-power:SUPER-SOT3
- removed R11, R12, R13, R14, R15, R16: (no value), rcl:R1206
- added IC3: 74AUC1G06DBV, 74xx-little-us:SOT23-5
- added IC4: 74AHC1G08DBV, 74xx-little-de:SOT23-5
- added IC6: 74AHC1G86DBV, 74xx-little-us:SOT23-5
- added R1: (no value), rcl:R1206
Connections:
- removed net A+: Q19.1, Q22.2, R14.2
- removed net B+: Q19.2
- removed net ENABLE: Q18.1, R15.2
- removed net N$35: Q22.1, R13.2
- removed net N$37: Q19.3, Q20.2
- removed net N$38: Q20.3
- removed net N$39: Q21.3
- removed net N$40: Q17.3, Q21.2, R11.1
- removed net N$41: Q17.1, Q22.3, R12.2
- removed net N$42: Q18.3, Q20.1, Q21.1, R16.1
- new net N$2: IC2.4, R1.1
- new net N$3: IC3.2, IC6.2
- new net N$6: IC3.4, IC4.1
- new net N$8: IC4.2, IC6.1
- net +5V: no longer R11.2, R16.2
- net 0V: no longer Q17.2, Q18.2, R12.1, R13.1, R14.1, R15.1
- net GND: now also IC3.3, IC4.3, IC6.3
- net OUT0: now also R1.2
- net VCC: now also IC3.5, IC4.5, IC6.5

Commit message: changed v2
Parts:
- removed C12, C13, C21: (no value), rcl:C1206
- removed D10: (no value), semicon-smd-ipc:SOD123
- removed Q23, Q24, Q25, Q26, Q62, Q63, Q64: FDN360P, transistor-power:SUPER-SOT3
- removed Q65, Q66: BSS123, transistor-small-signal:SOT23
- removed R53, R54, R55, R56, R57: (no value), rcl:R1206
- added C1, C8: (no value), rcl:C1206
- added IC10, IC11, IC12, IC13, IC14, IC15, IC16, IC18, IC20, IC7, IC8, IC9: 74LVC1G125DBV, 74xx-little-de:SOT23-5
- added IC17: 74AUC1G06DBV, 74xx-little-us:SOT23-5
- added IC19: 74AHC1G14DCK, 74xx-little-de:SC70-5
- added IC21: 74AHC1G08DBV, 74xx-little-de:SOT23-5
- added IC22: 74AHC1G86DBV, 74xx-little-us:SOT23-5
- added Q1, Q2, Q3, Q4: FDN360P, transistor-power:SUPER-SOT3
- added R10, R12, R2, R3, R6, R7, R8, R9: (no value), rcl:R1206
- IC3: value 74AUC1G06DBV -> 74LVC1G125DBV; device 74xx-little-us:SOT23-5 -> 74xx-little-de:SOT23-5
- IC4: value 74AHC1G08DBV -> 74LVC1G125DBV
- IC5: value 74AHC1G14DCK -> 74LVC1G125DBV; device 74xx-little-de:SC70-5 -> 74xx-little-de:SOT23-5
- IC6: value 74AHC1G86DBV -> 74LVC1G125DBV; device 74xx-little-us:SOT23-5 -> 74xx-little-de:SOT23-5
- Q10: value FDN360P -> BSS123; device transistor-power:SUPER-SOT3 -> transistor-small-signal:SOT23
- Q6: value BSS123 -> FDN360P; device transistor-small-signal:SOT23 -> transistor-power:SUPER-SOT3
- moved IC4 169.2 mm to (130.8, 30.5), turned to 90 degrees
- moved IC6 142.6 mm to (94.0, 30.5), turned to 90 degrees
- moved R4 113.4 mm to (147.3, 30.5), turned to 90 degrees
- moved IC2 107.6 mm to (85.1, 30.5), turned to 90 degrees
- moved R5 101.8 mm to (121.9, 16.5), turned to 90 degrees
- moved Q5 96.1 mm to (8.89, 76.2), turned to 90 degrees
- moved Q9 82.1 mm to (8.89, 54.6), turned to 90 degrees
- moved Q7 81.7 mm to (8.89, 66.0), turned to 90 degrees
- moved IC3 78.0 mm to (39.4, 30.5), turned to 90 degrees
- moved R1 76.5 mm to (50.8, 20.3), turned to 90 degrees
- moved Q8 71.0 mm to (8.89, 61.0), turned to 90 degrees
- moved Q6 65.6 mm to (8.89, 71.1), turned to 90 degrees
- moved IC5 55.1 mm to (69.8, 8.89), turned to 90 degrees
- moved C2 53.4 mm to (14.0, 90.2)
- moved IC1 51.8 mm to (36.8, 19.1)
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- renumbered R17 to R11
Connections:
- removed net N$3: IC3.2, IC6.2
- removed net N$49: Q63.3, Q64.2, R55.2
- removed net N$60: Q63.1, Q64.1, Q66.3, R56.1
- removed net N$61: C21.1, D10.1, Q66.1, R57.2
- removed net OUT_X2: D1.A, Q5.3
- new net N$10: IC16.4, R8.1
- new net N$11: IC3.4, IC7.2
- new net N$12: IC7.4, R3.1
- new net N$13: IC11.4, IC15.2
- new net N$14: IC15.4, R7.1
- new net N$15: IC2.4, IC6.2
- new net N$16: IC6.4, R2.1
- new net N$17: IC10.4, IC14.2
- new net N$18: IC14.4, R6.1
- new net N$19: IC4.4, IC8.2
- new net N$20: IC8.4, R4.1
- new net N$21: IC13.2, IC9.4
- new net N$22: IC13.4, R5.1
- new net N$23: IC18.4, IC20.2
- new net N$9: IC12.4, IC16.2
- new net OUT: R12.2
- new net X: IC20.1
- new net X_1: IC16.1
- new net X_2: IC7.1
- new net X_3: IC15.1
- new net X_4: IC6.1
- new net X_5: IC14.1
- new net X_6: IC8.1
- new net X_7: IC13.1
- new net Y_: D1.A, IC17.2, IC22.2, Q11.3
- net +5V: now also IC17.5, Q11.2; no longer Q5.2, Q62.2, R53.1, R56.2
- net 0V: now also C1.2, C8.2, IC17.3, Q10.2, R9.2; no longer C12.2, C13.2, C21.2, Q6.2, Q65.2, Q66.2, R4.2, R54.2, R57.1
- net A-Z: now also C11.1, IC19.2, Q1.3, Q2.3, Q3.3, Q4.3, Q5.3; no longer C9.1, IC5.2, Q11.3, Q23.3, Q24.3, Q25.3, Q26.3
- net CTR: now also IC10.1, IC11.1, IC12.1, IC18.1, IC2.1, IC21.4, IC3.1, IC4.1, IC9.1; no longer Q62.1, R53.2
- net DELTA: now also IC10.2, IC11.2, IC12.2, IC18.2, IC2.2, IC22.4, IC3.2, IC4.2, IC9.2; no longer Q65.1, R54.1
- net GND: now also IC10.3, IC11.3, IC12.3, IC13.3, IC14.3, IC15.3, IC16.3, IC18.3, IC19.3, IC20.3, IC21.3, IC22.3, IC7.3, IC8.3, IC9.3
- net N$1: now also IC5.2; no longer IC2.2
- net N$2: now also IC5.4; no longer IC2.4
- net N$24: now also IC20.4, R12.1; no longer Q62.3, Q65.3, R55.1
- net N$4: now also C10.1, Q10.1, R10.2, R9.1; no longer C2.1, Q6.1, R4.1, R5.2
- net N$5: now also R10.1; no longer R5.1
- net N$6: now also IC17.4, IC21.1; no longer IC3.4, IC4.1
- net N$7: now also IC19.4, Q11.1; no longer IC5.4, Q5.1
- net N$8: now also IC21.2, IC22.1; no longer IC4.2, IC6.1
- net OUT0: now also C1.1, Q1.1; no longer C13.1, Q26.1
- net OUT1: now also C2.1, Q2.1, R8.2; no longer C12.1, Q25.1
- net OUT2: now also C3.1, Q3.1, R3.2; no longer C11.1, Q24.1
- net OUT3: now also C4.1, Q4.1, R7.2; no longer C10.1, Q23.1
- net OUT4: now also Q5.1, R2.2; no longer Q9.1
- net OUT5: now also Q6.1, R6.2; no longer Q10.1
- net OUT6: now also C7.1, R4.2; no longer C3.1
- net OUT7: now also C8.1, R5.2; no longer C4.1
- net OUTX: now also C9.1, Q9.1; no longer C7.1, Q11.1, Q63.2, Q64.3
- net VCC: now also IC10.5, IC11.5, IC12.5, IC13.5, IC14.5, IC15.5, IC16.5, IC18.5, IC19.5, IC20.5, IC21.5, IC22.5, IC7.5, IC8.5, IC9.5
- net X0: now also Q1.2; no longer Q26.2
- net X1: now also Q2.2; no longer Q25.2
- net X2: now also Q3.2; no longer Q24.2
- net X3: now also Q4.2; no longer Q23.2
- net X4: now also Q5.2; no longer Q9.2
- net X5: now also Q6.2; no longer Q10.2
- net X_0: now also IC5.1; no longer IC2.1
- net X_X: now also Q9.2; no longer D10.2, Q11.2

Commit message: titelblatt + layout
Parts:
- IC13: value 74LVC1G125DBV -> 74AHC1G86DBV; device 74xx-little-de:SOT23-5 -> 74xx-little-us:SOT23-5
- IC17: value 74AUC1G06DBV -> 74LVC1G125DBV; device 74xx-little-us:SOT23-5 -> 74xx-little-de:SOT23-5
- IC18: value 74LVC1G125DBV -> 74AHC1G14DCK; device 74xx-little-de:SOT23-5 -> 74xx-little-de:SC70-5
- IC19: value 74AHC1G14DCK -> 74LVC1G125DBV; device 74xx-little-de:SC70-5 -> 74xx-little-de:SOT23-5
- IC21: value 74AHC1G08DBV -> 74LVC1G125DBV
- IC22: value 74AHC1G86DBV -> 74LVC1G125DBV; device 74xx-little-us:SOT23-5 -> 74xx-little-de:SOT23-5
- IC7: value 74LVC1G125DBV -> 74AUC1G06DBV; device 74xx-little-de:SOT23-5 -> 74xx-little-us:SOT23-5
- IC8: value 74LVC1G125DBV -> 74AHC1G08DBV
- Q10: value BSS123 -> FDN360P; device transistor-small-signal:SOT23 -> transistor-power:SUPER-SOT3
- Q11: value FDN360P -> BSS123; device transistor-power:SUPER-SOT3 -> transistor-small-signal:SOT23
- moved R12 146.6 mm to (11.4, 77.5), turned to 0 degrees
- moved IC9 127.4 mm to (36.8, 81.3), turned to 270 degrees
- moved IC18 125.1 mm to (19.1, 77.5), turned to 270 degrees
- moved R4 111.9 mm to (47.0, 80.0), turned to 0 degrees
- moved IC4 107.8 mm to (41.9, 91.4), turned to 270 degrees
- moved IC20 105.1 mm to (41.9, 61.0), turned to 270 degrees
- moved Q11 95.5 mm to (15.2, 81.3), turned to 180 degrees
- moved IC8 95.3 mm to (44.5, 34.3)
- moved R5 95.0 mm to (47.0, 74.9), turned to 0 degrees
- moved IC14 89.7 mm to (36.8, 71.1), turned to 270 degrees
- moved SV1 87.7 mm to (83.8, 69.8), turned to 270 degrees
- moved R6 86.9 mm to (47.0, 69.8), turned to 0 degrees
- moved IC5 84.2 mm to (36.8, 86.4), turned to 270 degrees
- moved IC10 83.3 mm to (41.9, 81.3), turned to 270 degrees
- moved R2 80.9 mm to (47.0, 90.2), turned to 0 degrees
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Connections:
- removed net OUT: R12.2
- net +5V: now also IC7.5, Q10.2; no longer IC17.5, Q11.2
- net 0V: now also IC7.3, Q11.2, R11.2, R12.1; no longer IC17.3, Q10.2, R11.1, R9.2
- net A-Z: now also IC18.2, Q11.3, R12.2; no longer IC19.2, Q10.3, R11.2
- net CTR: now also IC14.1, IC16.1, IC19.1, IC21.1, IC5.1, IC8.4; no longer IC10.1, IC12.1, IC18.1, IC2.1, IC21.4, IC4.1
- net DELTA: now also IC13.4, IC14.2, IC16.2, IC19.2, IC21.2, IC5.2; no longer IC10.2, IC12.2, IC18.2, IC2.2, IC22.4, IC4.2
- net GND: now also IC17.3; no longer IC7.3
- net N$1: now also IC3.4, IC4.2; no longer IC1.4, IC5.2
- net N$10: now also IC6.4, R3.1; no longer IC16.4, R8.1
- net N$11: now also IC10.2, IC9.4; no longer IC3.4, IC7.2
- net N$12: now also IC10.4, R4.1; no longer IC7.4, R3.1
- net N$13: now also IC12.2; no longer IC15.2
- net N$14: now also IC12.4, R5.1; no longer IC15.4, R7.1
- net N$15: now also IC14.4, IC15.2; no longer IC2.4, IC6.2
- net N$16: now also IC15.4, R6.1; no longer IC6.4, R2.1
- net N$17: now also IC16.4, IC17.2; no longer IC10.4, IC14.2
- net N$18: now also IC17.4, R7.1; no longer IC14.4, R6.1
- net N$19: now also IC19.4, IC20.2; no longer IC4.4, IC8.2
- net N$2: now also IC4.4, R2.1; no longer IC5.4, R1.1
- net N$20: now also IC20.4, R9.1; no longer IC8.4, R4.1
- net N$21: now also IC21.4, IC22.2; no longer IC13.2, IC9.4
- net N$22: now also IC22.4, R10.1; no longer IC13.4, R5.1
- net N$23: now also IC1.4, IC2.2; no longer IC18.4, IC20.2
- net N$24: now also IC2.4, R1.1; no longer IC20.4, R12.1
- net N$4: now also Q11.1, R11.1, R8.2; no longer Q10.1, R10.2, R9.1
- net N$5: now also R8.1; no longer R10.1
- net N$6: now also IC7.4, IC8.1; no longer IC17.4, IC21.1
- net N$7: now also IC18.4, Q10.1; no longer IC19.4, Q11.1
- net N$8: now also IC13.1, IC8.2; no longer IC21.2, IC22.1
- net N$9: now also IC5.4, IC6.2; no longer IC12.4, IC16.2
- net OUT0: now also C2.1, Q2.1, R2.2; no longer C1.1, Q1.1, R1.2
- net OUT1: now also C3.1, Q3.1, R3.2; no longer C2.1, Q2.1, R8.2
- net OUT2: now also C4.1, Q4.1, R4.2; no longer C3.1, Q3.1, R3.2
- net OUT3: now also C5.1, Q5.1, R5.2; no longer C4.1, Q4.1, R7.2
- net OUT4: now also C6.1, Q6.1, R6.2; no longer C5.1, Q5.1, R2.2
- net OUT5: now also C7.1, Q7.1, R7.2; no longer C6.1, Q6.1, R6.2
- net OUT6: now also C8.1, Q8.1, R9.2; no longer C7.1, Q7.1, R4.2
- net OUT7: now also C9.1, Q9.1, R10.2; no longer C8.1, Q8.1, R5.2
- net OUTX: now also C1.1, Q1.1, R1.2; no longer C9.1, Q9.1
- net VCC: now also IC17.5; no longer IC7.5
- net X: now also IC2.1; no longer IC20.1
- net X0: now also Q2.2; no longer Q1.2
- net X1: now also Q3.2; no longer Q2.2
- net X2: now also Q4.2; no longer Q3.2
- net X3: now also Q5.2; no longer Q4.2
- net X4: now also Q6.2; no longer Q5.2
- net X5: now also Q7.2; no longer Q6.2
- net X6: now also Q8.2; no longer Q7.2
- net X7: now also Q9.2; no longer Q8.2
- net X_0: now also IC4.1; no longer IC5.1
- net X_1: now also IC6.1; no longer IC16.1
- net X_2: now also IC10.1; no longer IC7.1
- net X_3: now also IC12.1; no longer IC15.1
- net X_4: now also IC15.1; no longer IC6.1
- net X_5: now also IC17.1; no longer IC14.1
- net X_6: now also IC20.1; no longer IC8.1
- net X_7: now also IC22.1; no longer IC13.1
- net X_X: now also Q1.2; no longer Q9.2
- net Y_: now also IC13.2, IC7.2, Q10.3; no longer IC17.2, IC22.2, Q11.3
Routing:
- net 0V: track 0.00 -> 186.1 mm, vias 0 -> 4
- net A-Z: track 0.00 -> 176.3 mm
- net VCC: track 0.00 -> 162.7 mm, vias 0 -> 3
- net GND: track 0.00 -> 161.2 mm, vias 0 -> 3
- net CTR: track 0.00 -> 87.6 mm, vias 0 -> 5
- net DELTA: track 0.00 -> 76.5 mm, vias 0 -> 4
- net Y_: track 0.00 -> 50.1 mm
- net +5V: track 0.00 -> 47.3 mm
- net X1: track 0.00 -> 35.7 mm
- net X7: track 0.00 -> 34.3 mm
- net X0: track 0.00 -> 30.2 mm
- net X3: track 0.00 -> 28.6 mm
- net X2: track 0.00 -> 27.1 mm, vias 0 -> 1
- net X5: track 0.00 -> 26.8 mm
- net X6: track 0.00 -> 26.6 mm
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
Commit message: malik aar und eagle
Parts:
- removed IC18: 74AHC1G14DCK, 74xx-little-de:SC70-5
- added C12: (no value), rcl:C1206
- added D2, D3: PMLL41SOD80C, diode:SOD80C
- added Q12: BSS123, transistor-small-signal:SOT23
- added Q13: BCX71SMD, transistor-pnp:SOT23
- added R13, R14, R15, R16, R17, R18: (no value), rcl:R1206
- added T1, T2, T3: BC846, transistor:SOT23
- Q10: value FDN360P -> BSS123; device transistor-power:SUPER-SOT3 -> transistor-small-signal:SOT23
- moved D1 119.8 mm to (2.54, -38.1)
- moved Q10 101.7 mm to (2.54, -24.1)
- moved R8 97.4 mm to (2.54, -8.89), turned to 0 degrees
Connections:
- new net N$3: C12.2, Q10.1, R8.1
- net +5V: now also R13.1, R14.1; no longer Q10.2
- net 0V: now also Q10.2, Q12.2, R8.2
- net A-Z: no longer IC18.2
- net GND: no longer IC18.3
- net N$4: now also D1.A, Q12.3, R14.2; no longer R8.2
- net N$5: now also Q10.3, Q12.1, R13.2; no longer D1.C, R8.1
- net N$7: now also C12.1; no longer IC18.4, Q10.1
- net VCC: no longer IC18.5
- net Y_: now also D1.C; no longer D1.A, Q10.3
Routing:
- net N$7: track 5.79 -> 0.00 mm
- net N$5: track 5.46 -> 0.00 mm
- net Y_: track 50.1 -> 45.3 mm

Commit message: überarbeitet
Parts:
- removed IC1, IC10, IC11, IC12, IC14, IC15, IC16, IC17, IC19, IC2, IC20, IC21, IC22, IC3, IC4, IC5, IC6, IC9: 74LVC1G125DBV, 74xx-little-de:SOT23-5
- removed IC13: 74AHC1G86DBV, 74xx-little-us:SOT23-5
- removed IC7: 74AUC1G06DBV, 74xx-little-us:SOT23-5
- removed IC8: 74AHC1G08DBV, 74xx-little-de:SOT23-5
- removed R10, R9: (no value), rcl:R1206
- added C13, C14, C15, C16, C17: (no value), rcl:C1206
- added D4, D5, D6, D7, D8: PMLL41SOD80C, diode:SOD80C
- added Q14, Q15, Q16, Q17, Q18, Q19, Q20, Q21, Q23, Q24, Q25, Q27, Q28, Q29, Q31, Q32, Q33, Q35, Q36, Q37, Q39, Q40, Q41: BSS123, transistor-small-signal:SOT23
- added Q22, Q26, Q30, Q34, Q38: BCX71SMD, transistor-pnp:SOT23
- added R19, R20, R21, R22, R23, R24, R25, R26, R27, R28, R29, R30, R31, R32, R33, R34, R35, R36, R37, R38, R39, R40, R41, R42, R43, R44, R45, R46, R47, R48, R49, R50, R51: (no value), rcl:R1206
- added T4, T5, T6, T7, T8: BC846, transistor:SOT23
- moved R2 488.9 mm to (12.7, -397.5)
- moved R3 483.5 mm to (17.8, -397.5)
- moved R4 478.1 mm to (22.9, -397.5)
- moved R6 474.5 mm to (2.54, -402.6)
- moved R7 469.0 mm to (7.62, -402.6)
- moved R5 466.9 mm to (19.1, -391.2)
- moved R1 448.8 mm to (7.62, -397.5)
Connections:
- net N$7 renamed OPV_OUT
- net OUTX renamed OUT_X
- removed net CTR: IC1.1, IC11.1, IC14.1, IC16.1, IC19.1, IC21.1, IC3.1, IC5.1, IC8.4, IC9.1
- removed net GND: IC1.3, IC10.3, IC11.3, IC12.3, IC13.3, IC14.3, IC15.3, IC16.3, IC17.3, IC19.3, IC2.3, IC20.3, IC21.3, IC22.3, IC3.3, IC4.3, IC5.3, IC6.3, IC8.3, IC9.3
- removed net N$13: IC11.4, IC12.2
- removed net N$14: IC12.4, R5.1
- removed net N$15: IC14.4, IC15.2
- removed net N$16: IC15.4, R6.1
- removed net N$17: IC16.4, IC17.2
- removed net N$18: IC17.4, R7.1
- removed net N$19: IC19.4, IC20.2
- removed net N$20: IC20.4, R9.1
- removed net N$21: IC21.4, IC22.2
- removed net N$22: IC22.4, R10.1
- removed net N$23: IC1.4, IC2.2
- removed net N$24: IC2.4, R1.1
- removed net OUT0: C2.1, Q2.1, R2.2
- removed net OUT1: C3.1, Q3.1, R3.2
- removed net OUT2: C4.1, Q4.1, R4.2
- removed net OUT3: C5.1, Q5.1, R5.2
- removed net OUT4: C6.1, Q6.1, R6.2
- removed net OUT5: C7.1, Q7.1, R7.2
- removed net OUT6: C8.1, Q8.1, R9.2
- removed net OUT7: C9.1, Q9.1, R10.2
- removed net VCC: IC1.5, IC10.5, IC11.5, IC12.5, IC13.5, IC14.5, IC15.5, IC16.5, IC17.5, IC19.5, IC2.5, IC20.5, IC21.5, IC22.5, IC3.5, IC4.5, IC5.5, IC6.5, IC8.5, IC9.5
- removed net X: IC2.1
- removed net X_4: IC15.1
- removed net X_5: IC17.1
- removed net X_6: IC20.1
- removed net X_7: IC22.1
- new net B: Q16.1, Q21.1
- new net EN: Q17.3, R21.1
- new net ENABLE: Q23.1, Q27.1, Q31.1, Q35.1, Q39.1, R28.2, R35.2, R42.2, R49.2, R5.2
- new net N$25: R17.1, T3.2
- new net N$26: Q13.1, R15.2, T2.3
- new net N$27: T1.2, T2.2, T3.3
- new net N$28: Q29.3, R32.1, T5.1
- new net N$29: D2.A, R16.2, T3.1
- new net N$30: Q14.3, Q15.1, R19.1
- new net N$31: D4.A, Q22.3
- new net N$32: Q15.2, Q16.3
- new net N$33: Q26.2, R31.1, T5.3
- new net N$34: Q22.1, R26.2
- new net N$35: Q23.3, Q25.1, R26.1, R27.1
- new net N$36: Q18.1, Q19.3, R22.1
- new net N$37: Q19.1, Q21.3, R23.1
- new net N$38: D5.A, Q26.3
- new net N$39: Q26.1, R33.2
- new net N$40: Q17.2, Q18.3
- new net N$41: Q27.3, Q29.1, R33.1, R34.1
- new net N$42: Q27.2, Q28.3
- new net N$43: Q19.2, Q20.3
- new net N$44: Q33.3, R39.1, T6.1
- new net N$45: Q30.2, R38.1, T6.3
- new net N$46: D6.A, Q30.3
- new net N$47: Q30.1, R40.2
- new net N$48: Q31.3, Q33.1, R40.1, R41.1
- new net N$49: Q31.2, Q32.3
- new net N$50: Q37.3, R46.1, T7.1
- new net N$51: Q34.2, R45.1, T7.3
- new net N$52: D7.A, Q34.3
- new net N$53: Q34.1, R47.2
- new net N$54: Q35.3, Q37.1, R47.1, R48.1
- new net N$55: Q35.2, Q36.3
- new net N$7: Q23.2, Q24.3
- new net OP_OUT: Q13.3, R18.1
- new net OUT_0: C2.1, Q2.1, R24.2
- new net OUT_1: C3.1, Q3.1, R31.2
- new net OUT_2: C4.1, Q4.1, R45.2
- new net OUT_3: C5.1, Q5.1, R38.2
- new net OUT_4: C6.1, Q6.1
- new net OUT_5: C7.1, Q7.1
- new net OUT_6: C8.1, Q8.1
- new net OUT_7: C9.1, Q9.1
- net +5V: now also Q13.2, R15.1, R16.1, R19.2, R2.2, R20.2, R21.2, R22.2, R23.2, R25.2, R27.2, R32.2, R34.2, R39.2, R4.2, R41.2, R46.2, R48.2, T1.1, T1.3; no longer IC7.5
- net 0V: now also C13.2, C14.2, C15.2, C16.2, C17.2, D3.C, Q14.2, Q16.2, Q18.2, Q20.2, Q21.2, Q24.2, Q25.2, Q28.2, Q29.2, Q32.2, Q33.2, Q36.2, Q37.2, Q40.2, Q41.2, R17.2, R18.2, R28.1, R29.1, R30.1, R35.1, R36.1, R37.1, R42.1, R43.1, R44.1, R49.1, R5.1, R50.1, R51.1, R6.1, R7.1; no longer IC7.3
- net A-Z: now also T2.1
- net DELTA: now also D4.C, D5.C, D6.C, D7.C, D8.C, Q15.3, Q17.1, R20.1, T4.2, T5.2, T6.2, T7.2, T8.2; no longer IC1.2, IC11.2, IC13.4, IC14.2, IC16.2, IC19.2, IC21.2, IC3.2, IC5.2, IC9.2
- net N$1: now also Q41.3, R2.1, T8.1; no longer IC3.4, IC4.2
- net N$10: now also Q38.1, R3.2; no longer IC6.4, R3.1
- net N$11: now also Q39.3, Q41.1, R3.1, R4.1; no longer IC10.2, IC9.4
- net N$12: now also Q39.2, Q40.3; no longer IC10.4, R4.1
- net N$2: now also Q38.2, R1.1, T8.3; no longer IC4.4, R2.1
- net N$6: now also Q25.3, R25.1, T4.1; no longer IC7.4, IC8.1
- net N$8: now also Q22.2, R24.1, T4.3; no longer IC13.1, IC8.2
- net N$9: now also D8.A, Q38.3; no longer IC5.4, IC6.2
- net X_0: now also C13.1, Q24.1, R29.2, R30.2; no longer IC4.1
- net X_1: now also C14.1, Q28.1, R36.2, R37.2; no longer IC6.1
- net X_2: now also C16.1, Q36.1, R50.2, R51.2; no longer IC10.1
- net X_3: now also C15.1, Q32.1, R43.2, R44.2; no longer IC12.1
- net X_X: now also C17.1, Q40.1, R6.2, R7.2
- net Y_: now also Q14.1, Q20.1; no longer IC13.2, IC7.2
Routing:
- net CTR: track 87.6 -> 0.00 mm, vias 5 -> 0
- net DELTA: track 76.5 -> 0.00 mm, vias 4 -> 0
- net +5V: track 47.2 -> 0.00 mm
- net Y_: track 45.3 -> 0.00 mm
- net OUT4: track 14.0 -> 0.00 mm
- net OUT7: track 14.0 -> 0.00 mm
- net OUT1: track 14.0 -> 0.00 mm
- net OUT6: track 14.0 -> 0.00 mm
- net OUT3: track 14.0 -> 0.00 mm
- net OUT0: track 14.0 -> 0.00 mm
- net OUT5: track 13.9 -> 0.00 mm
- net OUT2: track 13.9 -> 0.00 mm
- net OUT_6: track 0.00 -> 13.9 mm
- net OUT_3: track 0.00 -> 13.9 mm
- net OUT_0: track 0.00 -> 13.9 mm
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
Commit message: layout angepasst
Parts:
- moved R47 456.0 mm to (12.7, 90.2), turned to 90 degrees
- moved D7 455.4 mm to (29.2, 95.2), turned to 180 degrees
- moved R45 455.2 mm to (29.2, 88.9)
- moved R46 454.7 mm to (19.1, 88.9), turned to 90 degrees
- moved R48 454.7 mm to (16.5, 88.9), turned to 90 degrees
- moved R50 443.8 mm to (24.1, 72.4), turned to 90 degrees
- moved R51 443.4 mm to (19.1, 72.4), turned to 90 degrees
- moved C16 438.6 mm to (21.6, 72.4), turned to 270 degrees
- moved Q34 437.4 mm to (24.1, 92.7)
- moved T7 436.9 mm to (24.1, 85.1)
- moved R1 436.7 mm to (63.5, 35.6)
- moved R3 436.6 mm to (47.0, 38.1), turned to 90 degrees
- moved D8 436.1 mm to (63.5, 40.6), turned to 180 degrees
- moved R2 435.1 mm to (54.6, 35.6), turned to 90 degrees
- moved R4 434.1 mm to (52.1, 35.6), turned to 90 degrees
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Connections:
- removed net OP_OUT: Q13.3, R18.1
- new net N$13: D2.C, D3.A
- net OPV_OUT: now also Q13.3, R18.1
Routing:
- net +5V: track 0.00 -> 377.6 mm, vias 0 -> 7
- net 0V: track 185.9 -> 497.2 mm, vias 4 -> 7
- net DELTA: track 0.00 -> 226.8 mm, vias 0 -> 2
- net VCC: track 162.7 -> 0.00 mm, vias 3 -> 0
- net GND: track 161.2 -> 0.00 mm, vias 3 -> 0
- net ENABLE: track 0.00 -> 136.9 mm, vias 0 -> 4
- net A-Z: track 176.0 -> 111.2 mm
- net Y_: track 0.00 -> 54.2 mm, vias 0 -> 2
- net N$4: track 15.4 -> 66.4 mm, vias 0 -> 2
- net OUT_2: track 3.22 -> 49.2 mm, vias 0 -> 3
- net X_X: track 0.00 -> 40.1 mm, vias 0 -> 2
- net OUT_3: track 13.9 -> 44.7 mm, vias 0 -> 2
- net OPV_OUT: track 0.00 -> 21.5 mm
- net B: track 0.00 -> 20.4 mm
- net N$48: track 0.00 -> 19.8 mm
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Other:
- board size 160 x 100 mm -> 127 x 100 mm

Commit message: Eagle Korrektur
(Nur oberflächlich)
Parts:
- removed C6, C7, C8, C9: (no value), rcl:C1206
- removed Q6, Q7, Q8, Q9: FDN360P, transistor-power:SUPER-SOT3
Connections:
- removed net OUT_4: C6.1, Q6.1
- removed net OUT_5: C7.1, Q7.1
- removed net OUT_6: C8.1, Q8.1
- removed net OUT_7: C9.1, Q9.1
- net 0V: no longer C6.2, C7.2, C8.2, C9.2
- net A-Z: no longer Q6.3, Q7.3, Q8.3, Q9.3
- net X4: no longer Q6.2
- net X5: no longer Q7.2
- net X6: no longer Q8.2
- net X7: no longer Q9.2
Routing:
- net 0V: track 497.2 -> 0.00 mm, vias 7 -> 0
- net A-Z: track 111.2 -> 0.00 mm
- net X7: track 31.2 -> 0.00 mm
- net X5: track 26.7 -> 0.00 mm
- net X6: track 26.4 -> 0.00 mm
- net X4: track 23.9 -> 0.00 mm
- net OUT_6: track 2.74 -> 0.00 mm
- net OUT_5: track 2.72 -> 0.00 mm
- net OUT_4: track 2.71 -> 0.00 mm
- net OUT_7: track 2.70 -> 0.00 mm
