File: Eagle Projekt/Hardware-Neuron v2/Hardware-Neuron.brd (EAGLE design)
At the start: 127 x 100 mm, 116 parts, among them Q1 FDN360P, Q10 BSS123, Q11 BSS123, Q12 BSS123, Q13 BCX71SMD, Q14 BSS123, Q15 BSS123, Q16 BSS123, Q17 BSS123, Q18 BSS123, Q19 BSS123, Q2 FDN360P, Q20 BSS123, Q21 BSS123, Q22 BCX71SMD, Q23 BSS123, Q24 BSS123, Q25 BSS123, Q26 BCX71SMD, Q27 BSS123, Q28 BSS123, Q29 BSS123, Q3 FDN360P, Q30 BCX71SMD, Q31 BSS123, Q32 BSS123, Q33 BSS123, Q34 BCX71SMD, Q35 BSS123, Q36 BSS123, Q37 BSS123, Q38 BCX71SMD, Q39 BSS123, Q4 FDN360P, Q40 BSS123, Q41 BSS123, Q5 FDN360P, T1 BC846, T2 BC846, T3 BC846, T4 BC846, T5 BC846, T6 BC846, T7 BC846, T8 BC846

Commit message: Cosmetics
Eagle Kontrolliert, Dokumente geortnet
Parts:
- added R10, R9: (no value), rcl:R1206
Connections:
- new net N$14: R10.1, R9.2, T1.1
- net +5V: now also C17.1, Q40.1, R6.2, R7.2, R9.1; no longer T1.1
- net 0V: now also R10.2
- net X_X: no longer C17.1, Q40.1, R6.2, R7.2
Routing:
- net X_X: track 40.1 -> 34.3 mm
- net +5V: track 377.6 -> 382.7 mm
Changed lines of the file:
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@@
 <attribute name="NAME" x="52.705" y="31.115" size="1.27" layer="25"/>
+</element>
+<element name="R9" library="rcl" library_urn="urn:adsk.eagle:library:334" package="R1206" package3d_urn="urn:adsk.eagle:package:23540/2" value="" x="2.54" y="-3.81">
+<attribute name="SPICEPREFIX" value="R" x="2.54" y="-3.81" size="1.778" layer="27" display="off"/>
+</element>
+<element name="R10" library="rcl" library_urn="urn:adsk.eagle:library:334" package="R1206" package3d_urn="urn:adsk.eagle:package:23540/2" value="" x="2.54" y="-10.16">
+<attribute name="SPICEPREFIX" value="R" x="2.54" y="-10.16" size="1.778" layer="27" display="off"/>
 </element>
 </elements>
@@
 <contactref element="R27" pad="2"/>
 <contactref element="R25" pad="2"/>
-<contactref element="T1" pad="1"/>
 <contactref element="R34" pad="2"/>
 <contactref element="R32" pad="2"/>
@@
 <wire x1="74.041" y1="26.8224" x2="74.041" y2="25.7048" width="0.4064" layer="1"/>
 <wire x1="74.8792" y1="27.6606" x2="74.041" y2="26.8224" width="0.4064" layer="1"/>
-<wire x1="74.041" y1="25.7048" x2="73.98" y2="25.57" width="0.4064" layer="1"/>
 <wire x1="74.8792" y1="27.6606" x2="74.93" y2="27.77" width="0.4064" layer="1"/>
 <wire x1="81.3054" y1="34.3662" x2="85.217" y2="34.3662" width="0.4064" layer="1"/>
@@
 <wire x1="89.1286" y1="26.543" x2="89.1286" y2="18.7198" width="0.4064" layer="1"/>
 <wire x1="87.7316" y1="27.94" x2="89.1286" y2="26.543" width="0.4064" layer="1"/>
-<wire x1="74.041" y1="25.4254" x2="73.98" y2="25.57" width="0.4064" layer="1"/>
 <wire x1="87.7316" y1="27.94" x2="87.63" y2="28.092" width="0.4064" layer="1"/>
 <wire x1="89.408" y1="39.3954" x2="101.4222" y2="39.3954" width="0.4064" layer="1"/>
@@
 <via x="111.2012" y="90.5256" extent="1-16" drill="0.35"/>
 <via x="113.157" y="43.5864" extent="1-16" drill="0.35"/>
+<contactref element="Q40" pad="1"/>
+<contactref element="R7" pad="2"/>
+<contactref element="C17" pad="1"/>
+<contactref element="R6" pad="2"/>
+<wire x1="54.483" y1="23.1902" x2="52.2478" y2="23.1902" width="0.4064" layer="1"/>
+<wire x1="52.2478" y1="23.1902" x2="52.07" y2="23.012" width="0.4064" layer="1"/>
+<wire x1="54.483" y1="23.1902" x2="54.61" y2="23.012" width="0.4064" layer="1"/>
+<wire x1="56.9976" y1="23.1902" x2="54.7624" y2="23.1902" width="0.4064" layer="1"/>
+<wire x1="54.7624" y1="23.1902" x2="54.61" y2="23.012" width="0.4064" layer="1"/>
+<wire x1="56.9976" y1="23.1902" x2="57.15" y2="22.99" width="0.4064" layer="1"/>
+<contactref element="R9" pad="1"/>
+<wire x1="74.041" y1="25.4254" x2="74.041" y2="25.7048" width="0" layer="19" extent="1-1"/>
+<wire x1="61.28" y1="25.57" x2="74.041" y2="25.7048" width="0" layer="19" extent="1-1"/>
+<wire x1="57.15" y1="22.99" x2="61.28" y2="25.57" width="0" layer="19" extent="1-1"/>
+<wire x1="1.118" y1="-3.81" x2="52.07" y2="23.012" width="0" layer="19" extent="1-1"/>
 </signal>
 <signal name="0V">
@@
 <contactref element="R7" pad="1"/>
 <contactref element="C17" pad="2"/>
+<contactref element="R10" pad="2"/>
 <wire x1="115.25" y1="75.1" x2="122.87" y2="75.1" width="0" layer="19" extent="1-1"/>
 <wire x1="108.9" y1="81.45" x2="115.25" y2="75.1" width="0" layer="19" extent="1-1"/>
@@
 <wire x1="72.52" y1="88.9" x2="72.52" y2="83.82" width="0" layer="19" extent="1-1"/>
 <wire x1="72.52" y1="73.66" x2="72.52" y2="78.74" width="0" layer="19" extent="1-1"/>
+<wire x1="3.962" y1="-10.16" x2="46.99" y2="22.708" width="0" layer="19" extent="1-1"/>
 </signal>
 <signal name="N$4">
@@
 <contactref element="R12" pad="2"/>
 <contactref element="C11" pad="1"/>
+<contactref element="Q11" pad="3"/>
+<contactref element="T2" pad="1"/>
+<contactref element="Q2" pad="3"/>
+<contactref element="Q1" pad="3"/>
+<contactref element="Q3" pad="3"/>
 <contactref element="Q4" pad="3"/>
 <contactref element="Q5" pad="3"/>
-<contactref element="Q3" pad="3"/>
-<contactref element="Q2" pad="3"/>
-<contactref element="Q11" pad="3"/>
-<contactref element="T2" pad="1"/>
-<contactref element="Q1" pad="3"/>
 <wire x1="64.94" y1="85.09" x2="64.94" y2="90.17" width="0" layer="19" extent="1-1"/>
 <wire x1="64.94" y1="80.01" x2="64.94" y2="85.09" width="0" layer="19" extent="1-1"/>
@@
 <signal name="X_X">
 <contactref element="Q1" pad="2"/>
-<contactref element="Q40" pad="1"/>
-<contactref element="R7" pad="2"/>
-<contactref element="C17" pad="1"/>
-<contactref element="R6" pad="2"/>
-<wire x1="54.483" y1="23.1902" x2="52.2478" y2="23.1902" width="0.4064" layer="1"/>
-<wire x1="52.2478" y1="23.1902" x2="52.07" y2="23.012" width="0.4064" layer="1"/>
-<wire x1="54.483" y1="23.1902" x2="54.61" y2="23.012" width="0.4064" layer="1"/>
 <wire x1="60.071" y1="25.4254" x2="61.1886" y2="25.4254" width="0.4064" layer="1"/>
 <wire x1="57.8358" y1="23.1902" x2="59.9313" y2="25.2857" width="0.4064" layer="1"/>
 <wire x1="59.9313" y1="25.2857" x2="60.071" y2="25.4254" width="0.4064" layer="1"/>
 <wire x1="57.277" y1="23.1902" x2="57.8358" y2="23.1902" width="0.4064" layer="1"/>
-<wire x1="61.1886" y1="25.4254" x2="61.28" y2="25.57" width="0.4064" layer="1"/>
-<wire x1="57.277" y1="23.1902" x2="57.15" y2="22.99" width="0.4064" layer="1"/>
 <wire x1="65.659" y1="50.5714" x2="67.056" y2="50.5714" width="0.4064" layer="1"/>
 <wire x1="65.659" y1="30.734" x2="65.659" y2="50.5714" width="0.4064" layer="16"/>
@@
 <wire x1="67.056" y1="50.5714" x2="67.14" y2="50.48" width="0.4064" layer="1"/>
 <wire x1="60.071" y1="25.146" x2="59.9313" y2="25.2857" width="0.4064" layer="1"/>
-<wire x1="56.9976" y1="23.1902" x2="54.7624" y2="23.1902" width="0.4064" layer="1"/>
-<wire x1="54.7624" y1="23.1902" x2="54.61" y2="23.012" width="0.4064" layer="1"/>
-<wire x1="56.9976" y1="23.1902" x2="57.15" y2="22.99" width="0.4064" layer="1"/>
 <via x="65.659" y="50.5714" extent="1-16" drill="0.35"/>
 <via x="60.071" y="25.146" extent="1-16" drill="0.35"/>
@@
 <wire x1="87.7316" y1="15.9258" x2="87.63" y2="16.08" width="0.4064" layer="1"/>
 </signal>
+<signal name="N$14">
+<contactref element="R9" pad="2"/>
+<contactref element="T1" pad="1"/>
+<contactref element="R10" pad="1"/>
+<wire x1="3.962" y1="-3.81" x2="73.98" y2="25.57" width="0" layer="19" extent="1-1"/>
+<wire x1="1.118" y1="-10.16" x2="3.962" y2="-3.81" width="0" layer="19" extent="1-1"/>
+</signal>
 </signals>
