File: Eagle Projekt/Hardware-Neuron v2/Hardware-Neuron.brd (EAGLE design)
At the start: 127 x 100 mm, 118 parts, among them Q1 FDN360P, Q10 BSS123, Q11 BSS123, Q12 BSS123, Q13 BCX71SMD, Q14 BSS123, Q15 BSS123, Q16 BSS123, Q17 BSS123, Q18 BSS123, Q19 BSS123, Q2 FDN360P, Q20 BSS123, Q21 BSS123, Q22 BCX71SMD, Q23 BSS123, Q24 BSS123, Q25 BSS123, Q26 BCX71SMD, Q27 BSS123, Q28 BSS123, Q29 BSS123, Q3 FDN360P, Q30 BCX71SMD, Q31 BSS123, Q32 BSS123, Q33 BSS123, Q34 BCX71SMD, Q35 BSS123, Q36 BSS123, Q37 BSS123, Q38 BCX71SMD, Q39 BSS123, Q4 FDN360P, Q40 BSS123, Q41 BSS123, Q5 FDN360P, T1 BC846, T2 BC846, T3 BC846, T4 BC846, T5 BC846, T6 BC846, T7 BC846, T8 BC846

Commit message: dimensionierung
Parts:
- C1, C11, C2, C3, C4, C5: value (none) -> 10n
- C12, C13, C14, C15, C16, C17: value (none) -> 100n
- R1: value (none) -> 10M
- R11, R12, R13, R14, R2, R3, R4, R5, R6, R7, R8: value (none) -> 1k
- R24, R31, R38, R45: value (none) -> 10ME
- R25, R26, R27, R28, R29, R30, R32, R33, R34, R35, R36, R37, R39, R40, R41, R42, R43, R44, R46, R47, R48, R49, R50, R51: value (none) -> 1kE
- moved R9 63.5 mm to (62.2, 17.8), turned to 90 degrees
- moved R10 58.5 mm to (54.6, 16.5), turned to 180 degrees
Routing:
- net 0V: track 0.00 -> 511.3 mm, vias 0 -> 4
- net A-Z: track 0.00 -> 131.1 mm, vias 0 -> 5
- net +5V: track 382.7 -> 343.6 mm, vias 7 -> 9
- net X_X: track 34.3 -> 0.00 mm, vias 2 -> 0
- net DELTA: track 226.8 -> 254.6 mm, vias 2 -> 3
- net N$14: track 0.00 -> 21.7 mm
- net ENABLE: track 136.9 -> 143.1 mm
- net OUT_3: track 44.7 -> 50.5 mm, vias 2 -> 0
- net N$55: track 7.03 -> 10.6 mm
- net OUT_2: track 49.2 -> 50.6 mm, vias 3 -> 2
- net X2: track 28.4 -> 27.1 mm, vias 0 -> 1
- net OUT_X: track 16.6 -> 17.9 mm
- net X3: track 29.7 -> 28.6 mm
- net OUT_1: vias 2 -> 0
Other:
- board size 127 x 100 mm -> 127 x 98.7 mm

Commit message: dimensionierung
Parts:
- C10: value (none) -> 10n
- R10, R15, R16, R17, R18, R19, R20, R21, R22, R23, R9: value (none) -> 1k
Connections:
- removed net X_X: Q1.2
- net +5V: now also Q1.2
Changed lines of the file:
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@@
 <attribute name="VALUE" x="69.85" y="86.36" size="1.27" layer="27"/>
 </element>
-<element name="C10" library="rcl" library_urn="urn:adsk.eagle:library:334" package="C1206" package3d_urn="urn:adsk.eagle:package:23618/2" value="" x="67.31" y="6.35" smashed="yes">
+<element name="C10" library="rcl" library_urn="urn:adsk.eagle:library:334" package="C1206" package3d_urn="urn:adsk.eagle:package:23618/2" value="10n" x="67.31" y="6.35" smashed="yes">
 <attribute name="NAME" x="68.58" y="5.08" size="1.27" layer="25" rot="R180"/>
 <attribute name="SPICEPREFIX" value="C" x="102.87" y="-55.88" size="1.778" layer="27" display="off"/>
@@
 <attribute name="VALUE" x="83.185" y="23.495" size="1.27" layer="27" rot="R180"/>
 </element>
-<element name="R15" library="rcl" library_urn="urn:adsk.eagle:library:334" package="R1206" package3d_urn="urn:adsk.eagle:package:23540/2" value="" x="81.28" y="33.02" smashed="yes" rot="R270">
+<element name="R15" library="rcl" library_urn="urn:adsk.eagle:library:334" package="R1206" package3d_urn="urn:adsk.eagle:package:23540/2" value="1k" x="81.28" y="33.02" smashed="yes" rot="R270">
 <attribute name="NAME" x="82.55" y="34.29" size="1.27" layer="25" rot="R270"/>
 <attribute name="SPICEPREFIX" value="R" x="81.28" y="33.02" size="1.778" layer="27" rot="R270" display="off"/>
 <attribute name="VALUE" x="78.74" y="34.29" size="1.27" layer="27" rot="R270"/>
 </element>
-<element name="R16" library="rcl" library_urn="urn:adsk.eagle:library:334" package="R1206" package3d_urn="urn:adsk.eagle:package:23540/2" value="" x="87.63" y="26.67" smashed="yes" rot="R270">
+<element name="R16" library="rcl" library_urn="urn:adsk.eagle:library:334" package="R1206" package3d_urn="urn:adsk.eagle:package:23540/2" value="1k" x="87.63" y="26.67" smashed="yes" rot="R270">
 <attribute name="NAME" x="88.9" y="27.94" size="1.27" layer="25" rot="R270"/>
 <attribute name="SPICEPREFIX" value="R" x="87.63" y="26.67" size="1.778" layer="27" rot="R270" display="off"/>
 <attribute name="VALUE" x="85.09" y="27.94" size="1.27" layer="27" rot="R270"/>
 </element>
-<element name="R17" library="rcl" library_urn="urn:adsk.eagle:library:334" package="R1206" package3d_urn="urn:adsk.eagle:package:23540/2" value="" x="81.28" y="12.7" smashed="yes" rot="R270">
+<element name="R17" library="rcl" library_urn="urn:adsk.eagle:library:334" package="R1206" package3d_urn="urn:adsk.eagle:package:23540/2" value="1k" x="81.28" y="12.7" smashed="yes" rot="R270">
 <attribute name="NAME" x="82.55" y="13.97" size="1.27" layer="25" rot="R270"/>
 <attribute name="SPICEPREFIX" value="R" x="81.28" y="12.7" size="1.778" layer="27" rot="R270" display="off"/>
 <attribute name="VALUE" x="78.74" y="13.97" size="1.27" layer="27" rot="R270"/>
 </element>
-<element name="R18" library="rcl" library_urn="urn:adsk.eagle:library:334" package="R1206" package3d_urn="urn:adsk.eagle:package:23540/2" value="" x="91.44" y="16.51" smashed="yes" rot="R270">
+<element name="R18" library="rcl" library_urn="urn:adsk.eagle:library:334" package="R1206" package3d_urn="urn:adsk.eagle:package:23540/2" value="1k" x="91.44" y="16.51" smashed="yes" rot="R270">
 <attribute name="NAME" x="92.71" y="17.78" size="1.27" layer="25" rot="R270"/>
 <attribute name="SPICEPREFIX" value="R" x="91.44" y="16.51" size="1.778" layer="27" rot="R270" display="off"/>
@@
 <attribute name="NAME" x="106.045" y="62.865" size="1.27" layer="25"/>
 </element>
-<element name="R19" library="rcl" library_urn="urn:adsk.eagle:library:334" package="R1206" package3d_urn="urn:adsk.eagle:package:23540/2" value="" x="107.95" y="88.9" smashed="yes" rot="R90">
+<element name="R19" library="rcl" library_urn="urn:adsk.eagle:library:334" package="R1206" package3d_urn="urn:adsk.eagle:package:23540/2" value="1k" x="107.95" y="88.9" smashed="yes" rot="R90">
 <attribute name="NAME" x="106.68" y="87.63" size="1.27" layer="25" rot="R90"/>
 <attribute name="SPICEPREFIX" value="R" x="107.95" y="88.9" size="1.778" layer="27" rot="R90" display="off"/>
 <attribute name="VALUE" x="110.49" y="87.63" size="1.27" layer="27" rot="R90"/>
 </element>
-<element name="R20" library="rcl" library_urn="urn:adsk.eagle:library:334" package="R1206" package3d_urn="urn:adsk.eagle:package:23540/2" value="" x="114.3" y="88.9" smashed="yes" rot="R90">
+<element name="R20" library="rcl" library_urn="urn:adsk.eagle:library:334" package="R1206" package3d_urn="urn:adsk.eagle:package:23540/2" value="1k" x="114.3" y="88.9" smashed="yes" rot="R90">
 <attribute name="NAME" x="113.03" y="87.63" size="1.27" layer="25" rot="R90"/>
 <attribute name="SPICEPREFIX" value="R" x="114.3" y="88.9" size="1.778" layer="27" rot="R90" display="off"/>
 <attribute name="VALUE" x="116.84" y="87.63" size="1.27" layer="27" rot="R90"/>
 </element>
-<element name="R21" library="rcl" library_urn="urn:adsk.eagle:library:334" package="R1206" package3d_urn="urn:adsk.eagle:package:23540/2" value="" x="121.92" y="88.9" smashed="yes" rot="R90">
+<element name="R21" library="rcl" library_urn="urn:adsk.eagle:library:334" package="R1206" package3d_urn="urn:adsk.eagle:package:23540/2" value="1k" x="121.92" y="88.9" smashed="yes" rot="R90">
 <attribute name="NAME" x="120.65" y="87.63" size="1.27" layer="25" rot="R90"/>
 <attribute name="SPICEPREFIX" value="R" x="121.92" y="88.9" size="1.778" layer="27" rot="R90" display="off"/>
 <attribute name="VALUE" x="124.46" y="87.63" size="1.27" layer="27" rot="R90"/>
 </element>
-<element name="R22" library="rcl" library_urn="urn:adsk.eagle:library:334" package="R1206" package3d_urn="urn:adsk.eagle:package:23540/2" value="" x="114.3" y="68.58" smashed="yes" rot="R270">
+<element name="R22" library="rcl" library_urn="urn:adsk.eagle:library:334" package="R1206" package3d_urn="urn:adsk.eagle:package:23540/2" value="1k" x="114.3" y="68.58" smashed="yes" rot="R270">
 <attribute name="NAME" x="115.57" y="69.85" size="1.27" layer="25" rot="R270"/>
 <attribute name="SPICEPREFIX" value="R" x="114.3" y="68.58" size="1.778" layer="27" rot="R270" display="off"/>
 <attribute name="VALUE" x="111.76" y="69.85" size="1.27" layer="27" rot="R270"/>
 </element>
-<element name="R23" library="rcl" library_urn="urn:adsk.eagle:library:334" package="R1206" package3d_urn="urn:adsk.eagle:package:23540/2" value="" x="107.95" y="68.58" smashed="yes" rot="R270">
+<element name="R23" library="rcl" library_urn="urn:adsk.eagle:library:334" package="R1206" package3d_urn="urn:adsk.eagle:package:23540/2" value="1k" x="107.95" y="68.58" smashed="yes" rot="R270">
 <attribute name="NAME" x="109.22" y="69.85" size="1.27" layer="25" rot="R270"/>
 <attribute name="SPICEPREFIX" value="R" x="107.95" y="68.58" size="1.778" layer="27" rot="R270" display="off"/>
@@
 <attribute name="NAME" x="52.705" y="31.115" size="1.27" layer="25"/>
 </element>
-<element name="R9" library="rcl" library_urn="urn:adsk.eagle:library:334" package="R1206" package3d_urn="urn:adsk.eagle:package:23540/2" value="" x="62.23" y="17.78" smashed="yes" rot="R90">
+<element name="R9" library="rcl" library_urn="urn:adsk.eagle:library:334" package="R1206" package3d_urn="urn:adsk.eagle:package:23540/2" value="1k" x="62.23" y="17.78" smashed="yes" rot="R90">
 <attribute name="NAME" x="60.96" y="16.51" size="1.27" layer="25" rot="R90"/>
 <attribute name="SPICEPREFIX" value="R" x="62.23" y="17.78" size="1.778" layer="27" rot="R90" display="off"/>
 <attribute name="VALUE" x="64.77" y="16.51" size="1.27" layer="27" rot="R90"/>
 </element>
-<element name="R10" library="rcl" library_urn="urn:adsk.eagle:library:334" package="R1206" package3d_urn="urn:adsk.eagle:package:23540/2" value="" x="54.61" y="16.51" smashed="yes" rot="R180">
+<element name="R10" library="rcl" library_urn="urn:adsk.eagle:library:334" package="R1206" package3d_urn="urn:adsk.eagle:package:23540/2" value="1k" x="54.61" y="16.51" smashed="yes" rot="R180">
 <attribute name="NAME" x="55.88" y="15.24" size="1.27" layer="25" rot="R180"/>
 <attribute name="SPICEPREFIX" value="R" x="54.61" y="16.51" size="1.778" layer="27" rot="R180" display="off"/>
@@
 <via x="111.2012" y="56.7182" extent="1-16" drill="0.35"/>
 <via x="76.5556" y="31.2928" extent="1-16" drill="0.35"/>
+<contactref element="Q1" pad="2"/>
+<wire x1="67.14" y1="50.48" x2="60.6298" y2="47.2186" width="0" layer="19" extent="1-16"/>
 </signal>
 <signal name="0V">
@@
 <wire x1="92.4814" y1="73.4822" x2="92.71" y2="73.66" width="0.4064" layer="1"/>
 </signal>
-<signal name="X_X">
-<contactref element="Q1" pad="2"/>
-</signal>
 <signal name="DELTA">
