File: Eagle Projekt/Hardware-Neuron v2/Hardware-Neuron.sch (EAGLE design)
At the start: 54 parts, among them IC1 74LVC1G125DBV, IC2 74LVC1G125DBV, IC5 74AHC1G14DCK, Q10 FDN360P, Q11 FDN360P, Q17 BSS123, Q18 BSS123, Q19 FDN360P, Q20 FDN360P, Q21 FDN360P, Q22 FDN360P, Q23 FDN360P, Q24 FDN360P, Q25 FDN360P, Q26 FDN360P, Q5 FDN360P, Q6 BSS123, Q62 FDN360P, Q63 FDN360P, Q64 FDN360P, Q65 BSS123, Q66 BSS123, Q7 FDN360P, Q8 FDN360P, Q9 FDN360P

Commit message: updated v2
Parts:
- removed Q17, Q18: BSS123, transistor-small-signal:BSS123
- removed Q19, Q20, Q21, Q22: FDN360P, transistor-power:FDN360P
- removed R11, R12, R13, R14, R15, R16: (no value), rcl:R-EU_R1206
- added IC3: 74AUC1G06DBV, 74xx-little-us:74AUC1G06DBV
- added IC4: 74AHC1G08DBV, 74xx-little-de:74AHC1G08DBV
- added IC6: 74AHC1G86DBV, 74xx-little-us:74AHC1G86DBV
- added R1: (no value), rcl:R-EU_R1206
Connections:
- removed net A+: Q19.G, Q22.S, R14.2
- removed net B+: Q19.S
- removed net ENABLE: Q18.G, R15.2
- removed net N$35: Q22.G, R13.2
- removed net N$37: Q19.D, Q20.S
- removed net N$38: Q20.D
- removed net N$39: Q21.D
- removed net N$40: Q17.D, Q21.S, R11.1
- removed net N$41: Q17.G, Q22.D, R12.2
- removed net N$42: Q18.D, Q20.G, Q21.G, R16.1
- new net N$2: IC2A.O, R1.1
- new net N$3: IC3G$1.I, IC6A.I1
- new net N$6: IC3G$1.O, IC4A.I0
- new net N$8: IC4A.I1, IC6A.I0
- net +5V: no longer R11.2, R16.2
- net 0V: no longer Q17.S, Q18.S, R12.1, R13.1, R14.1, R15.1
- net OUT0: now also R1.2

Commit message: changed v2
Parts:
- removed C12, C21: (no value), rcl:C-EUC1206
- removed D10: (no value), semicon-smd-ipc:D-SOD123
- removed Q62, Q63, Q64: FDN360P, transistor-power:FDN360P
- removed Q65, Q66: BSS123, transistor-small-signal:BSS123
- removed R17, R53, R54, R55, R56, R57: (no value), rcl:R-EU_R1206
- added C8: (no value), rcl:C-EUC1206
- added IC10, IC11, IC12, IC13, IC14, IC15, IC16, IC18, IC20, IC7, IC8, IC9: 74LVC1G125DBV, 74xx-little-de:74LVC1G125DBV
- added IC17: 74AUC1G06DBV, 74xx-little-us:74AUC1G06DBV
- added IC19: 74AHC1G14DCK, 74xx-little-de:74AHC1G14DCK
- added IC21: 74AHC1G08DBV, 74xx-little-de:74AHC1G08DBV
- added IC22: 74AHC1G86DBV, 74xx-little-us:74AHC1G86DBV
- added R10, R11, R12, R2, R3, R6, R7, R8, R9: (no value), rcl:R-EU_R1206
- IC3: value 74AUC1G06DBV -> 74LVC1G125DBV; device 74xx-little-us:74AUC1G06DBV -> 74xx-little-de:74LVC1G125DBV
- IC4: value 74AHC1G08DBV -> 74LVC1G125DBV; device 74xx-little-de:74AHC1G08DBV -> 74xx-little-de:74LVC1G125DBV
- IC5: value 74AHC1G14DCK -> 74LVC1G125DBV; device 74xx-little-de:74AHC1G14DCK -> 74xx-little-de:74LVC1G125DBV
- IC6: value 74AHC1G86DBV -> 74LVC1G125DBV; device 74xx-little-us:74AHC1G86DBV -> 74xx-little-de:74LVC1G125DBV
- Q10: value FDN360P -> BSS123; device transistor-power:FDN360P -> transistor-small-signal:BSS123
- Q6: value BSS123 -> FDN360P; device transistor-small-signal:BSS123 -> transistor-power:FDN360P
- renumbered C13 to C1, Q23 to Q4, Q24 to Q3, Q25 to Q2, Q26 to Q1
Connections:
- removed net N$3: IC3G$1.I, IC6A.I1
- removed net N$49: Q63.D, Q64.S, R55.2
- removed net N$60: Q63.G, Q64.G, Q66.D, R56.1
- removed net N$61: C21.1, D10.C, Q66.G, R57.2
- removed net OUT_X2: D1.A, Q5.D
- new net N$10: IC16A.O, R8.1
- new net N$11: IC3A.O, IC7A.I
- new net N$12: IC7A.O, R3.1
- new net N$13: IC11A.O, IC15A.I
- new net N$14: IC15A.O, R7.1
- new net N$15: IC2A.O, IC6A.I
- new net N$16: IC6A.O, R2.1
- new net N$17: IC10A.O, IC14A.I
- new net N$18: IC14A.O, R6.1
- new net N$19: IC4A.O, IC8A.I
- new net N$20: IC8A.O, R4.1
- new net N$21: IC13A.I, IC9A.O
- new net N$22: IC13A.O, R5.1
- new net N$23: IC18A.O, IC20A.I
- new net N$9: IC12A.O, IC16A.I
- new net OUT: R12.2
- new net X: IC20A.OE
- new net X_1: IC16A.OE
- new net X_2: IC7A.OE
- new net X_3: IC15A.OE
- new net X_4: IC6A.OE
- new net X_5: IC14A.OE
- new net X_6: IC8A.OE
- new net X_7: IC13A.OE
- new net Y_: D1.A, IC17G$1.I, IC22A.I1, Q11.D
- net +5V: now also IC17G$2.VCC, Q11.S; no longer Q5.S, Q62.S, R53.1, R56.2
- net 0V: now also C8.2, IC17G$2.GND, Q10.S, R11.1, R9.2; no longer C12.2, C21.2, Q6.S, Q65.S, Q66.S, R17.1, R4.2, R54.2, R57.1
- net A-Z: now also C11.1, IC19A.I, Q5.D, R11.2; no longer C9.1, IC5A.I, Q11.D, R17.2
- net CTR: now also IC10A.OE, IC11A.OE, IC12A.OE, IC18A.OE, IC21A.O, IC2A.OE, IC3A.OE, IC4A.OE, IC9A.OE; no longer Q62.G, R53.2
- net DELTA: now also IC10A.I, IC11A.I, IC12A.I, IC18A.I, IC22A.O, IC2A.I, IC3A.I, IC4A.I, IC9A.I; no longer Q65.G, R54.1
- net N$1: now also IC5A.I; no longer IC2A.I
- net N$2: now also IC5A.O; no longer IC2A.O
- net N$24: now also IC20A.O, R12.1; no longer Q62.D, Q65.D, R55.1
- net N$4: now also C10.1, Q10.G, R10.2, R9.1; no longer C2.1, Q6.G, R4.1, R5.2
- net N$5: now also R10.1; no longer R5.1
- net N$6: now also IC17G$1.O, IC21A.I0; no longer IC3G$1.O, IC4A.I0
- net N$7: now also IC19A.O, Q11.G; no longer IC5A.O, Q5.G
- net N$8: now also IC21A.I1, IC22A.I0; no longer IC4A.I1, IC6A.I0
- net OUT1: now also C2.1, R8.2; no longer C12.1
- net OUT2: now also C3.1, R3.2; no longer C11.1
- net OUT3: now also C4.1, R7.2; no longer C10.1
- net OUT4: now also Q5.G, R2.2; no longer Q9.G
- net OUT5: now also Q6.G, R6.2; no longer Q10.G
- net OUT6: now also C7.1, R4.2; no longer C3.1
- net OUT7: now also C8.1, R5.2; no longer C4.1
- net OUTX: now also C9.1, Q9.G; no longer C7.1, Q11.G, Q63.S, Q64.D
- net X4: now also Q5.S; no longer Q9.S
- net X5: now also Q6.S; no longer Q10.S
- net X_0: now also IC5A.OE; no longer IC2A.OE
- net X_X: now also Q9.S; no longer D10.A, Q11.S
Other:
- moved on the sheet: C10, C11, C2, C3, C4, C7, C9, D1, IC2, Q11, Q5, Q9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

Commit message: titelblatt + layout
Parts:
- IC13: value 74LVC1G125DBV -> 74AHC1G86DBV; device 74xx-little-de:74LVC1G125DBV -> 74xx-little-us:74AHC1G86DBV
- IC17: value 74AUC1G06DBV -> 74LVC1G125DBV; device 74xx-little-us:74AUC1G06DBV -> 74xx-little-de:74LVC1G125DBV
- IC18: value 74LVC1G125DBV -> 74AHC1G14DCK; device 74xx-little-de:74LVC1G125DBV -> 74xx-little-de:74AHC1G14DCK
- IC19: value 74AHC1G14DCK -> 74LVC1G125DBV; device 74xx-little-de:74AHC1G14DCK -> 74xx-little-de:74LVC1G125DBV
- IC21: value 74AHC1G08DBV -> 74LVC1G125DBV; device 74xx-little-de:74AHC1G08DBV -> 74xx-little-de:74LVC1G125DBV
- IC22: value 74AHC1G86DBV -> 74LVC1G125DBV; device 74xx-little-us:74AHC1G86DBV -> 74xx-little-de:74LVC1G125DBV
- IC7: value 74LVC1G125DBV -> 74AUC1G06DBV; device 74xx-little-de:74LVC1G125DBV -> 74xx-little-us:74AUC1G06DBV
- IC8: value 74LVC1G125DBV -> 74AHC1G08DBV; device 74xx-little-de:74LVC1G125DBV -> 74xx-little-de:74AHC1G08DBV
- Q10: value BSS123 -> FDN360P; device transistor-small-signal:BSS123 -> transistor-power:FDN360P
- Q11: value FDN360P -> BSS123; device transistor-power:FDN360P -> transistor-small-signal:BSS123
Connections:
- removed net OUT: R12.2
- net +5V: now also IC7G$2.VCC, Q10.S; no longer IC17G$2.VCC, Q11.S
- net 0V: now also IC7G$2.GND, Q11.S, R11.2, R12.1; no longer IC17G$2.GND, Q10.S, R11.1, R9.2
- net A-Z: now also IC18A.I, Q11.D, R12.2; no longer IC19A.I, Q10.D, R11.2
- net CTR: now also IC14A.OE, IC16A.OE, IC19A.OE, IC21A.OE, IC5A.OE, IC8A.O; no longer IC10A.OE, IC12A.OE, IC18A.OE, IC21A.O, IC2A.OE, IC4A.OE
- net DELTA: now also IC13A.O, IC14A.I, IC16A.I, IC19A.I, IC21A.I, IC5A.I; no longer IC10A.I, IC12A.I, IC18A.I, IC22A.O, IC2A.I, IC4A.I
- net N$1: now also IC3A.O, IC4A.I; no longer IC1A.O, IC5A.I
- net N$10: now also IC6A.O, R3.1; no longer IC16A.O, R8.1
- net N$11: now also IC10A.I, IC9A.O; no longer IC3A.O, IC7A.I
- net N$12: now also IC10A.O, R4.1; no longer IC7A.O, R3.1
- net N$13: now also IC12A.I; no longer IC15A.I
- net N$14: now also IC12A.O, R5.1; no longer IC15A.O, R7.1
- net N$15: now also IC14A.O, IC15A.I; no longer IC2A.O, IC6A.I
- net N$16: now also IC15A.O, R6.1; no longer IC6A.O, R2.1
- net N$17: now also IC16A.O, IC17A.I; no longer IC10A.O, IC14A.I
- net N$18: now also IC17A.O, R7.1; no longer IC14A.O, R6.1
- net N$19: now also IC19A.O, IC20A.I; no longer IC4A.O, IC8A.I
- net N$2: now also IC4A.O, R2.1; no longer IC5A.O, R1.1
- net N$20: now also IC20A.O, R9.1; no longer IC8A.O, R4.1
- net N$21: now also IC21A.O, IC22A.I; no longer IC13A.I, IC9A.O
- net N$22: now also IC22A.O, R10.1; no longer IC13A.O, R5.1
- net N$23: now also IC1A.O, IC2A.I; no longer IC18A.O, IC20A.I
- net N$24: now also IC2A.O, R1.1; no longer IC20A.O, R12.1
- net N$4: now also Q11.G, R11.1, R8.2; no longer Q10.G, R10.2, R9.1
- net N$5: now also R8.1; no longer R10.1
- net N$6: now also IC7G$1.O, IC8A.I0; no longer IC17G$1.O, IC21A.I0
- net N$7: now also IC18A.O, Q10.G; no longer IC19A.O, Q11.G
- net N$8: now also IC13A.I0, IC8A.I1; no longer IC21A.I1, IC22A.I0
- net N$9: now also IC5A.O, IC6A.I; no longer IC12A.O, IC16A.I
- net OUT0: now also C2.1, Q2.G, R2.2; no longer C1.1, Q1.G, R1.2
- net OUT1: now also C3.1, Q3.G, R3.2; no longer C2.1, Q2.G, R8.2
- net OUT2: now also C4.1, Q4.G, R4.2; no longer C3.1, Q3.G, R3.2
- net OUT3: now also C5.1, Q5.G, R5.2; no longer C4.1, Q4.G, R7.2
- net OUT4: now also C6.1, Q6.G, R6.2; no longer C5.1, Q5.G, R2.2
- net OUT5: now also C7.1, Q7.G, R7.2; no longer C6.1, Q6.G, R6.2
- net OUT6: now also C8.1, Q8.G, R9.2; no longer C7.1, Q7.G, R4.2
- net OUT7: now also C9.1, Q9.G, R10.2; no longer C8.1, Q8.G, R5.2
- net OUTX: now also C1.1, Q1.G, R1.2; no longer C9.1, Q9.G
- net X: now also IC2A.OE; no longer IC20A.OE
- net X0: now also Q2.S; no longer Q1.S
- net X1: now also Q3.S; no longer Q2.S
- net X2: now also Q4.S; no longer Q3.S
- net X3: now also Q5.S; no longer Q4.S
- net X4: now also Q6.S; no longer Q5.S
- net X5: now also Q7.S; no longer Q6.S
- net X6: now also Q8.S; no longer Q7.S
- net X7: now also Q9.S; no longer Q8.S
- net X_0: now also IC4A.OE; no longer IC5A.OE
- net X_1: now also IC6A.OE; no longer IC16A.OE
- net X_2: now also IC10A.OE; no longer IC7A.OE
- net X_3: now also IC12A.OE; no longer IC15A.OE
- net X_4: now also IC15A.OE; no longer IC6A.OE
- net X_5: now also IC17A.OE; no longer IC14A.OE
- net X_6: now also IC20A.OE; no longer IC8A.OE
- net X_7: now also IC22A.OE; no longer IC13A.OE
- net X_X: now also Q1.S; no longer Q9.S
- net Y_: now also IC13A.I1, IC7G$1.I, Q10.D; no longer IC17G$1.I, IC22A.I1, Q11.D
Other:
- moved on the sheet: C1, C2, C3, C4, C5, C6, C7, C8, C9, IC1, IC10, IC11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

Commit message: malik aar und eagle
Parts:
- removed IC18: 74AHC1G14DCK, 74xx-little-de:74AHC1G14DCK
- added C12: (no value), rcl:C-EUC1206
- added D2, D3: PMLL41SOD80C, diode:PMLL41SOD80C
- added Q12: BSS123, transistor-small-signal:BSS123
- added Q13: BCX71SMD, transistor-pnp:BCX71SMD
- added R13, R14, R15, R16, R17, R18: (no value), rcl:R-EU_R1206
- added T1, T2, T3: BC846, transistor:BC846
- Q10: value FDN360P -> BSS123; device transistor-power:FDN360P -> transistor-small-signal:BSS123
Connections:
- new net N$3: C12.2, Q10.G, R8.1
- net +5V: now also R13.1, R14.1; no longer Q10.S
- net 0V: now also Q10.S, Q12.S, R8.2
- net A-Z: no longer IC18A.I
- net N$4: now also D1.A, Q12.D, R14.2; no longer R8.2
- net N$5: now also Q10.D, Q12.G, R13.2; no longer D1.C, R8.1
- net N$7: now also C12.1; no longer IC18A.O, Q10.G
- net Y_: now also D1.C; no longer D1.A, Q10.D
Other:
- moved on the sheet: C10, C11, D1, Q11, R11, R12, R8

Commit message: überarbeitet
Parts:
- removed IC1, IC10, IC11, IC12, IC14, IC15, IC16, IC17, IC19, IC2, IC20, IC21, IC22, IC3, IC4, IC5, IC6, IC9: 74LVC1G125DBV, 74xx-little-de:74LVC1G125DBV
- removed IC13: 74AHC1G86DBV, 74xx-little-us:74AHC1G86DBV
- removed IC7: 74AUC1G06DBV, 74xx-little-us:74AUC1G06DBV
- removed IC8: 74AHC1G08DBV, 74xx-little-de:74AHC1G08DBV
- removed R10, R9: (no value), rcl:R-EU_R1206
- added C13, C14, C15, C16, C17: (no value), rcl:C-EUC1206
- added D4, D5, D6, D7, D8: PMLL41SOD80C, diode:PMLL41SOD80C
- added Q14, Q15, Q16, Q17, Q18, Q19, Q20, Q21, Q23, Q24, Q25, Q27, Q28, Q29, Q31, Q32, Q33, Q35, Q36, Q37, Q39, Q40, Q41: BSS123, transistor-small-signal:BSS123
- added Q22, Q26, Q30, Q34, Q38: BCX71SMD, transistor-pnp:BCX71SMD
- added R19, R20, R21, R22, R23, R24, R25, R26, R27, R28, R29, R30, R31, R32, R33, R34, R35, R36, R37, R38, R39, R40, R41, R42, R43, R44, R45, R46, R47, R48, R49, R50, R51: (no value), rcl:R-EU_R1206
- added T4, T5, T6, T7, T8: BC846, transistor:BC846
Connections:
- net N$7 renamed OPV_OUT
- net OUTX renamed OUT_X
- removed net CTR: IC11A.OE, IC14A.OE, IC16A.OE, IC19A.OE, IC1A.OE, IC21A.OE, IC3A.OE, IC5A.OE, IC8A.O, IC9A.OE
- removed net N$13: IC11A.O, IC12A.I
- removed net N$14: IC12A.O, R5.1
- removed net N$15: IC14A.O, IC15A.I
- removed net N$16: IC15A.O, R6.1
- removed net N$17: IC16A.O, IC17A.I
- removed net N$18: IC17A.O, R7.1
- removed net N$19: IC19A.O, IC20A.I
- removed net N$20: IC20A.O, R9.1
- removed net N$21: IC21A.O, IC22A.I
- removed net N$22: IC22A.O, R10.1
- removed net N$23: IC1A.O, IC2A.I
- removed net N$24: IC2A.O, R1.1
- removed net OUT0: C2.1, Q2.G, R2.2
- removed net OUT1: C3.1, Q3.G, R3.2
- removed net OUT2: C4.1, Q4.G, R4.2
- removed net OUT3: C5.1, Q5.G, R5.2
- removed net OUT4: C6.1, Q6.G, R6.2
- removed net OUT5: C7.1, Q7.G, R7.2
- removed net OUT6: C8.1, Q8.G, R9.2
- removed net OUT7: C9.1, Q9.G, R10.2
- removed net X: IC2A.OE
- removed net X_4: IC15A.OE
- removed net X_5: IC17A.OE
- removed net X_6: IC20A.OE
- removed net X_7: IC22A.OE
- new net B: Q16.G, Q21.G
- new net EN: Q17.D, R21.1
- new net ENABLE: Q23.G, Q27.G, Q31.G, Q35.G, Q39.G, R28.2, R35.2, R42.2, R49.2, R5.2
- new net N$25: R17.1, T3.E
- new net N$26: Q13.B, R15.2, T2.C
- new net N$27: T1.E, T2.E, T3.C
- new net N$28: Q29.D, R32.1, T5.B
- new net N$29: D2.A, R16.2, T3.B
- new net N$30: Q14.D, Q15.G, R19.1
- new net N$31: D4.A, Q22.C
- new net N$32: Q15.S, Q16.D
- new net N$33: Q26.E, R31.1, T5.C
- new net N$34: Q22.B, R26.2
- new net N$35: Q23.D, Q25.G, R26.1, R27.1
- new net N$36: Q18.G, Q19.D, R22.1
- new net N$37: Q19.G, Q21.D, R23.1
- new net N$38: D5.A, Q26.C
- new net N$39: Q26.B, R33.2
- new net N$40: Q17.S, Q18.D
- new net N$41: Q27.D, Q29.G, R33.1, R34.1
- new net N$42: Q27.S, Q28.D
- new net N$43: Q19.S, Q20.D
- new net N$44: Q33.D, R39.1, T6.B
- new net N$45: Q30.E, R38.1, T6.C
- new net N$46: D6.A, Q30.C
- new net N$47: Q30.B, R40.2
- new net N$48: Q31.D, Q33.G, R40.1, R41.1
- new net N$49: Q31.S, Q32.D
- new net N$50: Q37.D, R46.1, T7.B
- new net N$51: Q34.E, R45.1, T7.C
- new net N$52: D7.A, Q34.C
- new net N$53: Q34.B, R47.2
- new net N$54: Q35.D, Q37.G, R47.1, R48.1
- new net N$55: Q35.S, Q36.D
- new net N$7: Q23.S, Q24.D
- new net OP_OUT: Q13.C, R18.1
- new net OUT_0: C2.1, Q2.G, R24.2
- new net OUT_1: C3.1, Q3.G, R31.2
- new net OUT_2: C4.1, Q4.G, R45.2
- new net OUT_3: C5.1, Q5.G, R38.2
- new net OUT_4: C6.1, Q6.G
- new net OUT_5: C7.1, Q7.G
- new net OUT_6: C8.1, Q8.G
- new net OUT_7: C9.1, Q9.G
- net +5V: now also Q13.E, R15.1, R16.1, R19.2, R2.2, R20.2, R21.2, R22.2, R23.2, R25.2, R27.2, R32.2, R34.2, R39.2, R4.2, R41.2, R46.2, R48.2, T1.B, T1.C; no longer IC7G$2.VCC
- net 0V: now also C13.2, C14.2, C15.2, C16.2, C17.2, D3.C, Q14.S, Q16.S, Q18.S, Q20.S, Q21.S, Q24.S, Q25.S, Q28.S, Q29.S, Q32.S, Q33.S, Q36.S, Q37.S, Q40.S, Q41.S, R17.2, R18.2, R28.1, R29.1, R30.1, R35.1, R36.1, R37.1, R42.1, R43.1, R44.1, R49.1, R5.1, R50.1, R51.1, R6.1, R7.1; no longer IC7G$2.GND
- net A-Z: now also T2.B
- net DELTA: now also D4.C, D5.C, D6.C, D7.C, D8.C, Q15.D, Q17.G, R20.1, T4.E, T5.E, T6.E, T7.E, T8.E; no longer IC11A.I, IC13A.O, IC14A.I, IC16A.I, IC19A.I, IC1A.I, IC21A.I, IC3A.I, IC5A.I, IC9A.I
- net N$1: now also Q41.D, R2.1, T8.B; no longer IC3A.O, IC4A.I
- net N$10: now also Q38.B, R3.2; no longer IC6A.O, R3.1
- net N$11: now also Q39.D, Q41.G, R3.1, R4.1; no longer IC10A.I, IC9A.O
- net N$12: now also Q39.S, Q40.D; no longer IC10A.O, R4.1
- net N$2: now also Q38.E, R1.1, T8.C; no longer IC4A.O, R2.1
- net N$6: now also Q25.D, R25.1, T4.B; no longer IC7G$1.O, IC8A.I0
- net N$8: now also Q22.E, R24.1, T4.C; no longer IC13A.I0, IC8A.I1
- net N$9: now also D8.A, Q38.C; no longer IC5A.O, IC6A.I
- net X_0: now also C13.1, Q24.G, R29.2, R30.2; no longer IC4A.OE
- net X_1: now also C14.1, Q28.G, R36.2, R37.2; no longer IC6A.OE
- net X_2: now also C16.1, Q36.G, R50.2, R51.2; no longer IC10A.OE
- net X_3: now also C15.1, Q32.G, R43.2, R44.2; no longer IC12A.OE
- net X_X: now also C17.1, Q40.G, R6.2, R7.2
- net Y_: now also Q14.G, Q20.G; no longer IC13A.I1, IC7G$1.I
Other:
- note added: "Delta Calc"
- note added: "Komparator"
- note removed: "3StateVergleicherschaltung"
- note removed: "delta Apply"
- note removed: "delta Apply 0"
- note removed: "delta Apply 1"
- note removed: "delta Apply 2"
- note removed: "delta Apply 3"
- note removed: "delta Apply 4"
- note removed: "delta Apply 5"
- note removed: "delta Apply 6"
- note removed: "delta Apply 7"
- moved on the sheet: D2, D3, Q13, R1, R15, R16, R17, R18, R2, R3, R4, R5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

Commit message: layout angepasst
Connections:
- removed net OP_OUT: Q13.C, R18.1
- new net N$13: D2.C, D3.A
- net OPV_OUT: now also Q13.C, R18.1
Changed lines of the file:
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@@
 <label x="251.46" y="-68.58" size="1.778" layer="95"/>
+</segment>
+<segment>
+<pinref part="R18" gate="G$1" pin="1"/>
+<pinref part="Q13" gate="G$1" pin="C"/>
+<wire x1="373.38" y1="-71.12" x2="373.38" y2="-63.5" width="0.1524" layer="91"/>
+<wire x1="373.38" y1="-63.5" x2="373.38" y2="-55.88" width="0.1524" layer="91"/>
+<wire x1="373.38" y1="-63.5" x2="378.46" y2="-63.5" width="0.1524" layer="91"/>
+<junction x="373.38" y="-63.5"/>
+<label x="375.92" y="-63.5" size="1.778" layer="95"/>
 </segment>
 </net>
@@
 </segment>
 </net>
-<net name="OP_OUT" class="0">
-<segment>
-<pinref part="R18" gate="G$1" pin="1"/>
-<pinref part="Q13" gate="G$1" pin="C"/>
-<wire x1="373.38" y1="-71.12" x2="373.38" y2="-63.5" width="0.1524" layer="91"/>
-<wire x1="373.38" y1="-63.5" x2="373.38" y2="-55.88" width="0.1524" layer="91"/>
-<wire x1="373.38" y1="-63.5" x2="378.46" y2="-63.5" width="0.1524" layer="91"/>
-<junction x="373.38" y="-63.5"/>
-<label x="375.92" y="-63.5" size="1.778" layer="95"/>
-</segment>
-</net>
 <net name="N$30" class="0">
 <segment>
@@
 </segment>
 </net>
+<net name="N$13" class="0">
+<segment>
+<pinref part="D3" gate="G$1" pin="A"/>
+<pinref part="D2" gate="G$1" pin="C"/>
+<wire x1="365.76" y1="-86.36" x2="365.76" y2="-83.82" width="0.1524" layer="91"/>
+</segment>
+</net>

Commit message: Eagle Korrektur
(Nur oberflächlich)
Parts:
- removed C6, C7, C8, C9: (no value), rcl:C-EUC1206
- removed Q6, Q7, Q8, Q9: FDN360P, transistor-power:FDN360P
Connections:
- removed net OUT_4: C6.1, Q6.G
- removed net OUT_5: C7.1, Q7.G
- removed net OUT_6: C8.1, Q8.G
- removed net OUT_7: C9.1, Q9.G
- net 0V: no longer C6.2, C7.2, C8.2, C9.2
- net A-Z: no longer Q6.D, Q7.D, Q8.D, Q9.D
- net X4: no longer Q6.S
- net X5: no longer Q7.S
- net X6: no longer Q8.S
- net X7: no longer Q9.S
Other:
- moved on the sheet: C2, C3, C4, C5, Q2, Q3, Q4, Q5

Commit message: Cosmetics
Eagle Kontrolliert, Dokumente geortnet
Parts:
- added R10, R9: (no value), rcl:R-EU_R1206
Connections:
- new net N$14: R10.1, R9.2, T1.B
- net +5V: now also C17.1, Q40.G, R6.2, R7.2, R9.1; no longer T1.B
- net 0V: now also R10.2
- net X_X: no longer C17.1, Q40.G, R6.2, R7.2
Other:
- note added: "Delta Apply Bias"
- note added: "Delta Apply X0"
- note added: "Delta Apply X1"
- note added: "Delta Apply X2"
- note added: "Delta Apply X3"
- moved on the sheet: C1, C11, C13, C14, C15, C16, C2, C3, C4, C5, D2, D3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
