File: Eagle Projekt/Hardware-Neuron v4 mit 0805/Hardware-Neuron.sch (EAGLE design)
At the start: 118 parts, among them Q1 FDN360P, Q10 BSS123, Q11 BSS123, Q12 BSS123, Q13 FDN360P, Q14 BCX71SMD, Q15 BCX71SMD, Q16 BSS123, Q17 BSS123, Q18 BSS123, Q19 BSS123, Q2 BCX71SMD, Q20 BSS123, Q21 BSS123, Q22 BCX71SMD, Q23 BCX71SMD, Q24 BSS123, Q25 BSS123, Q26 BSS123, Q27 BSS123, Q28 BSS123, Q29 BSS123, Q3 BCX71SMD, Q30 BSS123, Q31 BSS123, Q32 BSS123, Q33 BSS123, Q34 BSS123, Q35 BSS123, Q36 BSS123, Q37 BSS123, Q4 FDN360P, Q5 FDN360P, Q6 BSS123, Q7 BSS123, Q8 BSS123, Q9 FDN360P, T1 BC846, T2 BC846, T3 BC846, T4 BC846, T5 BC846, T6 BC846, T7 BC846, T8 BC846

Commit message: Layout upgrade
Parts:
- removed C4: 10n, rcl:C-EUC1206
- removed C8: 100n, rcl:C-EUC1206
- removed D3: PMLL41SOD80C, diode:PMLL41SOD80C
- removed Q14: BCX71SMD, transistor-pnp:BCX71SMD
- removed Q16, Q18, Q20: BSS123, transistor-small-signal:BSS123
- removed Q9: FDN360P, transistor-power:FDN360P
- removed R15, R17, R18, R23, R25, R26: 1kE, rcl:R-EU_R1206
- removed R16: 10ME, rcl:R-EU_R1206
- removed T3: BC846, transistor:BC846
- C1, C10, C11, C12, C13, C2, C3, C5, C6, C7, C9: device rcl:C-EUC1206 -> rcl:C-EUC0805
- R1, R10, R11, R12, R13, R14, R19, R2, R20, R21, R22, R24, R27, R28, R29, R3, R30, R31, R32, R33, R34, R35, R36, R37, R38, R39, R4, R40, R41, R42, R43, R44, R45, R46, R47, R48, R49, R5, R50, R51, R6, R7, R8, R9: device rcl:R-EU_R1206 -> rcl:R-EU_M0805
Connections:
- removed net ENABLE: Q10.G, Q18.G, Q19.G, Q30.G, Q8.G, R10.2, R23.2, R24.2, R43.2, R9.2
- removed net N$44: Q16.D, R20.1, T3.B
- removed net N$45: Q14.E, R16.1, T3.C
- removed net N$46: D3.A, Q14.C
- removed net N$47: Q14.B, R15.2
- removed net N$48: Q16.G, Q18.D, R15.1, R21.1
- removed net N$49: Q18.S, Q20.D
- removed net OUT_3: C4.1, Q9.G, R16.2
- removed net X_3: C8.1, Q20.G, R25.2, R26.2
- net +5V: now also SV1.9; no longer R18.2, R19.2
- net 0V: now also SV1.10; no longer C4.2, C8.2, Q16.S, Q20.S, R23.1, R25.1, R26.1
- net A-Z: now also SV1.7; no longer Q9.D
- net DELTA: no longer D3.C, T3.E
- net EN: now also Q10.G, Q19.G, Q30.G, Q8.G, R10.2, R24.2, R43.2, R9.2, SV1.8
- net N$28: now also R21.1; no longer R19.1
- net N$39: now also R19.2; no longer R17.2
- net N$41: now also R19.1, R20.1; no longer R17.1, R18.1
- net X3: no longer Q9.S
Other:
- note removed: "Delta Apply X3"
- moved on the sheet: C10, C12, C13, D5, D6, D7, D8, Q22, Q23, Q24, Q25, Q26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
