File: Eagle Projekt/Hardware-Neuron v5 0v polygon/Hardware-Neuron.brd (EAGLE design)
At the start: 62.2 x 88.6 mm, 102 parts, among them Q1 FDN360P, Q10 BSS123, Q11 BSS123, Q12 BSS123, Q13 FDN360P, Q15 BCX71SMD, Q17 BSS123, Q19 BSS123, Q2 BCX71SMD, Q21 BSS123, Q22 BCX71SMD, Q23 BCX71SMD, Q24 BSS123, Q25 BSS123, Q26 BSS123, Q27 BSS123, Q28 BSS123, Q29 BSS123, Q3 BCX71SMD, Q30 BSS123, Q31 BSS123, Q32 BSS123, Q33 BSS123, Q34 BSS123, Q35 BSS123, Q36 BSS123, Q37 BSS123, Q4 FDN360P, Q5 FDN360P, Q6 BSS123, Q7 BSS123, Q8 BSS123, T1 BC846, T2 BC846, T4 BC846, T5 BC846, T6 BC846, T7 BC846, T8 BC846

Commit message: blä
Routing:
- net DELTA: track 191.7 -> 178.2 mm
- net EN: track 165.1 -> 176.6 mm, vias 5 -> 4
- net A-Z: track 88.6 -> 95.0 mm
- net Y_: track 99.1 -> 104.1 mm
- net +5V: track 337.1 -> 332.8 mm, vias 12 -> 9
- net OUT_2: track 56.8 -> 57.6 mm
- net X1: track 28.4 -> 29.1 mm
- net N$14: track 46.7 -> 46.8 mm, vias 2 -> 0
