File: Eagle Projekt/Hardware-Neuron v6/Hardware-Neuron.brd (EAGLE design)
At the start: 62.2 x 88.6 mm, 102 parts, among them Q1 FDN360P, Q10 BSS123, Q11 BSS123, Q12 BSS123, Q13 FDN360P, Q15 BCX71SMD, Q17 BSS123, Q19 BSS123, Q2 BCX71SMD, Q21 BSS123, Q22 BCX71SMD, Q23 BCX71SMD, Q24 BSS123, Q25 BSS123, Q26 BSS123, Q27 BSS123, Q28 BSS123, Q29 BSS123, Q3 BCX71SMD, Q30 BSS123, Q31 BSS123, Q32 BSS123, Q33 BSS123, Q34 BSS123, Q35 BSS123, Q36 BSS123, Q37 BSS123, Q4 FDN360P, Q5 FDN360P, Q6 BSS123, Q7 BSS123, Q8 BSS123, T1 BC846, T2 BC846, T4 BC846, T5 BC846, T6 BC846, T7 BC846, T8 BC846

Commit message: programming
Parts:
- moved C7 0.51 mm to (57.7, 68.3), flipped to the bottom, turned to 270 degrees
- moved C3 0.25 mm to (57.7, 73.7), flipped to the bottom
- moved Q1 0.25 mm to (54.1, 85.3), flipped to the bottom
- moved Q13 0.25 mm to (54.1, 70.1), flipped to the bottom
- moved Q4 0.25 mm to (54.1, 80.3), flipped to the bottom
- moved Q5 0.25 mm to (54.1, 75.2), flipped to the bottom
- flipped C1 to the bottom
- flipped C2 to the bottom
Routing:
- net 0V: track 415.6 -> 29.2 mm, vias 8 -> 0
- net +5V: track 9.22 -> 263.7 mm, vias 0 -> 3
- net OUT_2: track 56.8 -> 108.1 mm, vias 0 -> 1
- net DELTA: track 191.9 -> 142.7 mm, vias 5 -> 3
- net OUT_X: track 63.0 -> 81.1 mm, vias 2 -> 3
- net A-Z: track 88.6 -> 73.5 mm, vias 0 -> 1
- net Y_: track 99.1 -> 86.4 mm, vias 0 -> 2
- net OUT_0: track 18.9 -> 26.7 mm, vias 0 -> 1
- net EN: track 165.1 -> 158.6 mm, vias 5 -> 2
- net N$14: track 46.7 -> 52.4 mm
- net N$27: track 12.7 -> 17.0 mm
- net N$5: track 12.5 -> 16.7 mm
- net X2: track 26.5 -> 22.7 mm, vias 1 -> 0
- net N$16: track 32.4 -> 35.7 mm, vias 3 -> 0
- net B: track 72.6 -> 75.8 mm, vias 0 -> 4
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- added copper zone on layer 1, net 0V
- removed copper zone on layer 1, net +5V
