File: Eagle Projekt/Hardware-Neuron v7/Hardware-Neuron.brd (EAGLE design)
At the start: 62.2 x 88.6 mm, 102 parts, among them Q1 FDN360P, Q10 BSS123, Q11 BSS123, Q12 BSS123, Q13 FDN360P, Q15 BCX71SMD, Q17 BSS123, Q19 BSS123, Q2 BCX71SMD, Q21 BSS123, Q22 BCX71SMD, Q23 BCX71SMD, Q24 BSS123, Q25 BSS123, Q26 BSS123, Q27 BSS123, Q28 BSS123, Q29 BSS123, Q3 BCX71SMD, Q30 BSS123, Q31 BSS123, Q32 BSS123, Q33 BSS123, Q34 BSS123, Q35 BSS123, Q36 BSS123, Q37 BSS123, Q4 FDN360P, Q5 FDN360P, Q6 BSS123, Q7 BSS123, Q8 BSS123, T1 BC846, T2 BC846, T4 BC846, T5 BC846, T6 BC846, T7 BC846, T8 BC846

Commit message: stückliste und so
Parts:
- renumbered C12 to C8, C13 to C4, D8 to D5, Q33 to Q20, Q34 to Q18, Q35 to Q16, Q36 to Q14, Q37 to Q9, R45 to R26, R46 to R25, R47 to R23, R48 to R18, R49 to R17, R50 to R16, R51 to R15

Commit message: hu
Parts:
- removed Q24, Q26: BSS123, transistor-small-signal:SOT23
- removed R33, R41: 1k, rcl:M0805
- added Q33: BSS123, transistor-small-signal:SOT23
- added R45: 1k, rcl:M0805
- Q18, Q20: value BSS123 -> FDN360P; device transistor-small-signal:SOT23 -> transistor-power:SUPER-SOT3
- moved Q18 10.2 mm to (48.3, 3.81), turned to 0 degrees
- moved R4 7.73 mm to (29.2, 74.9)
- moved R6 7.73 mm to (36.8, 74.9)
- moved T2 7.73 mm to (41.9, 71.1)
- moved R5 7.73 mm to (33.0, 74.9)
- moved R15 7.62 mm to (20.3, 5.08)
- moved Q9 7.41 mm to (54.6, 6.35)
- moved D2 7.41 mm to (43.2, 77.5), turned to 270 degrees
- moved C3 6.84 mm to (55.1, 67.6)
- moved C7 6.84 mm to (55.1, 62.5)
- moved Q13 6.84 mm to (51.3, 63.8)
- moved C1 6.84 mm to (55.1, 77.7)
- moved C2 6.84 mm to (55.1, 72.6)
- moved Q1 6.84 mm to (51.3, 79.0)
- moved Q3 6.84 mm to (40.6, 77.5)
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Connections:
- removed net N$30: Q24.1, Q26.3, R33.1
- removed net N$37: Q18.1, Q20.3, R41.1
- removed net N$43: Q18.2, Q9.3
- new net N$17: Q18.3, Q9.3
- new net N$4: Q33.3, R45.1
- net +5V: now also R45.2; no longer R33.2, R41.2
- net 0V: now also Q33.2; no longer Q20.2, Q26.2
- net B: now also Q18.1; no longer Q20.1
- net DELTA: now also D1.A, D2.A, D3.A, D4.A, Q20.2, Q33.1; no longer D1.C, D2.C, D3.C, D4.C, Q24.3
- net N$31: now also D2.C; no longer D2.A
- net N$32: now also Q20.3; no longer Q24.2
- net N$36: now also Q18.2; no longer Q18.3
- net N$38: now also D4.C; no longer D4.A
- net N$52: now also D1.C; no longer D1.A
- net N$9: now also D3.C; no longer D3.A
- net Y_: now also Q20.1; no longer Q26.1
Routing:
- net +5V: track 340.1 -> 107.5 mm
- net Y_: track 117.4 -> 64.4 mm, vias 2 -> 1
- net A-Z: track 98.0 -> 63.3 mm
- net B: track 77.4 -> 62.7 mm
- net EN: track 176.7 -> 162.0 mm, vias 4 -> 2
- net OUT_2: track 57.6 -> 44.8 mm, vias 0 -> 2
- net N$32: track 3.27 -> 15.0 mm
- net N$37: track 11.1 -> 0.00 mm
- net DELTA: track 180.0 -> 169.3 mm, vias 5 -> 2
- net N$14: track 46.7 -> 36.8 mm
- net N$30: track 8.32 -> 0.00 mm
- net N$16: track 32.7 -> 40.8 mm, vias 3 -> 0
- net N$17: track 0.00 -> 7.77 mm, vias 0 -> 2
- net N$51: track 8.60 -> 16.0 mm
- net OUT_0: track 20.2 -> 15.3 mm, vias 0 -> 2
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- added copper zone on layer 16, net +5V
Other:
- board size 62.2 x 88.6 mm -> 59.7 x 82.2 mm

Commit message: jh
Parts:
- added 0V, EN, S, X0, X1, X2, Y_: PTR1PAD1-17, testpad:P1-17
- moved Q9 35.7 mm to (19.1, 8.89), turned to 180 degrees
- moved R42 31.8 mm to (15.2, 7.62), turned to 180 degrees
- moved Q33 30.7 mm to (3.81, 11.4)
- moved Q20 28.7 mm to (22.9, 14.0)
- moved Q27 27.9 mm to (15.2, 3.81)
- moved Q25 26.8 mm to (11.4, 11.4)
- moved R29 26.7 mm to (3.81, 5.08)
- moved Q18 26.7 mm to (21.6, 3.81)
- moved R45 26.7 mm to (10.2, 3.81)
- moved Q28 25.7 mm to (17.8, 12.7)
- moved R30 22.9 mm to (7.62, 8.89)
- moved D3 16.5 mm to (21.6, 38.1)
- moved Q23 16.5 mm to (16.5, 35.6)
- moved Q29 16.5 mm to (12.7, 27.9)
- moved Q30 16.5 mm to (8.89, 26.7)
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Connections:
- removed net B: Q18.1, Q27.1, SV1.5
- removed net X3: SV1.4
- new net S: Q18.1, Q27.1, S.TP, SV1.5
- net 0V: now also 0V.TP
- net EN: now also EN.TP
- net X0: now also X0.TP
- net X1: now also X1.TP
- net X2: now also X2.TP
- net Y_: now also Y_.TP
Routing:
- net S: track 0.00 -> 75.1 mm, vias 0 -> 1
- net B: track 62.7 -> 0.00 mm, vias 1 -> 0
- net Y_: track 64.4 -> 107.0 mm, vias 1 -> 0
- net N$14: track 36.8 -> 10.8 mm
- net X2: track 23.3 -> 43.7 mm
- net X0: track 37.0 -> 57.4 mm, vias 1 -> 0
- net A-Z: track 63.3 -> 80.1 mm, vias 1 -> 2
- net X1: track 27.5 -> 42.6 mm
- net OUT_2: track 44.8 -> 59.4 mm, vias 2 -> 0
- net OUT_X: track 65.7 -> 51.3 mm
- net DELTA: track 169.3 -> 156.9 mm
- net EN: track 162.0 -> 172.2 mm, vias 2 -> 4
- net N$32: track 15.0 -> 23.0 mm
- net 0V: track 0.00 -> 7.46 mm, vias 0 -> 1
- net N$51: track 16.0 -> 8.57 mm
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