File: Eagle Projekt/Hardware-Neuron v7/Hardware-Neuron.sch (EAGLE design)
At the start: 102 parts, among them Q1 FDN360P, Q10 BSS123, Q11 BSS123, Q12 BSS123, Q13 FDN360P, Q15 BCX71SMD, Q17 BSS123, Q19 BSS123, Q2 BCX71SMD, Q21 BSS123, Q22 BCX71SMD, Q23 BCX71SMD, Q24 BSS123, Q25 BSS123, Q26 BSS123, Q27 BSS123, Q28 BSS123, Q29 BSS123, Q3 BCX71SMD, Q30 BSS123, Q31 BSS123, Q32 BSS123, Q33 BSS123, Q34 BSS123, Q35 BSS123, Q36 BSS123, Q37 BSS123, Q4 FDN360P, Q5 FDN360P, Q6 BSS123, Q7 BSS123, Q8 BSS123, T1 BC846, T2 BC846, T4 BC846, T5 BC846, T6 BC846, T7 BC846, T8 BC846

Commit message: stückliste und so
Parts:
- renumbered C12 to C8, C13 to C4, D8 to D5, Q33 to Q20, Q34 to Q18, Q35 to Q16, Q36 to Q14, Q37 to Q9, R45 to R26, R46 to R25, R47 to R23, R48 to R18, R49 to R17, R50 to R16, R51 to R15

Commit message: hu
Parts:
- removed Q24, Q26: BSS123, transistor-small-signal:BSS123
- removed R33, R41: 1k, rcl:R-EU_M0805
- added Q33: BSS123, transistor-small-signal:BSS123
- added R45: 1k, rcl:R-EU_M0805
- Q18, Q20: value BSS123 -> FDN360P; device transistor-small-signal:BSS123 -> transistor-power:FDN360P
Connections:
- removed net N$30: Q24.G, Q26.D, R33.1
- removed net N$37: Q18.G, Q20.D, R41.1
- removed net N$43: Q18.S, Q9.D
- new net N$17: Q18.D, Q9.D
- new net N$4: Q33.D, R45.1
- net +5V: now also R45.2; no longer R33.2, R41.2
- net 0V: now also Q33.S; no longer Q20.S, Q26.S
- net B: now also Q18.G; no longer Q20.G
- net DELTA: now also D1.A, D2.A, D3.A, D4.A, Q20.S, Q33.G; no longer D1.C, D2.C, D3.C, D4.C, Q24.D
- net N$31: now also D2.C; no longer D2.A
- net N$32: now also Q20.D; no longer Q24.S
- net N$36: now also Q18.S; no longer Q18.D
- net N$38: now also D4.C; no longer D4.A
- net N$52: now also D1.C; no longer D1.A
- net N$9: now also D3.C; no longer D3.A
- net Y_: now also Q20.G; no longer Q26.G
Other:
- moved on the sheet: D1, D2, D3, D4

Commit message: jh
Parts:
- added 0V, EN, S, X0, X1, X2, Y_: PTR1PAD1-17, testpad:PTR1PAD1-17
Connections:
- removed net B: Q18.G, Q27.G, SV1.5
- removed net X3: SV1.4
- new net S: Q18.G, Q27.G, S.TP, SV1.5
- net 0V: now also 0V.TP
- net EN: now also EN.TP
- net X0: now also X0.TP
- net X1: now also X1.TP
- net X2: now also X2.TP
- net Y_: now also Y_.TP
Other:
- moved on the sheet: D6, D7, Q22, R15, R16, R25, R31, R37, R40, T5, T6, T8
